Commit message: Edit leader arm raw data to int 32

File: avatar_description/urdf/follower/follower.urdf.xacro (robot description, xacro)
@@ -42,3 +42,8 @@
     mock_sensor_commands="$(arg mock_sensor_commands)"
     port_name="$(arg port_name)"/>
+  <gazebo>
+    <plugin filename="libign_ros2_control-system.so" name="ign_ros2_control::IgnitionROS2ControlPlugin">
+      <parameters>$(find avatar_bringup)/config/follower/hardware_controller_manager.yaml</parameters>
+    </plugin>
+  </gazebo>
 </robot>

File: avatar_description/urdf/follower/follower_arm.urdf.xacro (robot description, xacro)
@@ -356,5 +356,5 @@
       <child link="right_link1_1"/>
       <axis xyz="-0.0 -1.0 0.0"/>
-      <limit velocity="4.8" effort="1000" lower="${-pi*2.0}" upper="${pi*2.0}" />
+      <limit velocity="4.8" effort="30" lower="${-pi*2.0}" upper="${pi*2.0}" />
       <dynamics damping="0.1" />
     </joint>
@@ -364,5 +364,5 @@
       <child link="right_link2_1"/>
       <axis xyz="-1.0 -0.0 0.0"/>
-      <limit velocity="4.8" effort="1000" lower="${-pi*2.0}" upper="${pi*2.0}" />
+      <limit velocity="4.8" effort="30" lower="${-pi*2.0}" upper="${pi*2.0}" />
       <dynamics damping="0.1" />
     </joint>
@@ -372,5 +372,5 @@
       <child link="right_link3_1"/>
       <axis xyz="0.0 -0.0 -1.0"/>
-      <limit velocity="4.8" effort="1000" lower="${-pi*2.0}" upper="${pi*2.0}" />
+      <limit velocity="4.8" effort="30" lower="${-pi*2.0}" upper="${pi*2.0}" />
       <dynamics damping="0.1" />
     </joint>
@@ -380,5 +380,5 @@
       <child link="right_link4_1"/>
       <axis xyz="0.0 1.0 -0.0"/>
-      <limit velocity="4.8" effort="1000" lower="${-pi*2.0}" upper="${pi*2.0}" />
+      <limit velocity="4.8" effort="30" lower="${-pi*2.0}" upper="${pi*2.0}" />
       <dynamics damping="0.1" />
     </joint>
@@ -388,5 +388,5 @@
       <child link="right_link5_1"/>
       <axis xyz="0.0 0.0 -1.0"/>
-      <limit velocity="4.8" effort="1000" lower="${-pi*2.0}" upper="${pi*2.0}" />
+      <limit velocity="4.8" effort="30" lower="${-pi*2.0}" upper="${pi*2.0}" />
       <dynamics damping="0.1" />
     </joint>
@@ -396,5 +396,5 @@
       <child link="right_link6_1"/>
       <axis xyz="0.0 1.0 0.0"/>
-      <limit velocity="4.8" effort="1000" lower="${-pi*2.0}" upper="${pi*2.0}" />
+      <limit velocity="4.8" effort="30" lower="${-pi*2.0}" upper="${pi*2.0}" />
       <dynamics damping="0.1" />
     </joint>
@@ -404,5 +404,5 @@
       <child link="right_link_gripper_1"/>
       <axis xyz="1.0 -0.0 -0.0"/>
-      <limit velocity="4.8" effort="1000" lower="${-pi*2.0}" upper="${pi*2.0}" />
+      <limit velocity="4.8" effort="30" lower="${-pi*2.0}" upper="${pi*2.0}" />
       <dynamics damping="0.1" />
     </joint>
@@ -412,5 +412,5 @@
       <child link="left_link1_1"/>
       <axis xyz="0.0 1.0 0.0"/>
-      <limit velocity="4.8" effort="1000" lower="${-pi*2.0}" upper="${pi*2.0}" />
+      <limit velocity="4.8" effort="30" lower="${-pi*2.0}" upper="${pi*2.0}" />
       <dynamics damping="0.1" />
     </joint>
@@ -420,5 +420,5 @@
       <child link="left_link2_1"/>
       <axis xyz="-1.0 -0.0 -0.0"/>
-      <limit velocity="4.8" effort="1000" lower="${-pi*2.0}" upper="${pi*2.0}" />
+      <limit velocity="4.8" effort="30" lower="${-pi*2.0}" upper="${pi*2.0}" />
       <dynamics damping="0.1" />
     </joint>
@@ -428,5 +428,5 @@
       <child link="left_link3_1"/>
       <axis xyz="0.0 -0.0 -1.0"/>
-      <limit velocity="4.8" effort="1000" lower="${-pi*2.0}" upper="${pi*2.0}" />
+      <limit velocity="4.8" effort="30" lower="${-pi*2.0}" upper="${pi*2.0}" />
       <dynamics damping="0.1" />
     </joint>
@@ -436,5 +436,5 @@
       <child link="left_link4_1"/>
       <axis xyz="-0.0 -1.0 0.0"/>
-      <limit velocity="4.8" effort="1000" lower="${-pi*2.0}" upper="${pi*2.0}" />
+      <limit velocity="4.8" effort="30" lower="${-pi*2.0}" upper="${pi*2.0}" />
       <dynamics damping="0.1" />
     </joint>
@@ -444,5 +444,5 @@
       <child link="left_link5_1"/>
       <axis xyz="0.0 0.0 -1.0"/>
-      <limit velocity="4.8" effort="1000" lower="${-pi*2.0}" upper="${pi*2.0}" />
+      <limit velocity="4.8" effort="30" lower="${-pi*2.0}" upper="${pi*2.0}" />
       <dynamics damping="0.1" />
     </joint>
@@ -452,5 +452,5 @@
       <child link="left_link6_1"/>
       <axis xyz="-0.0 -1.0 -0.0"/>
-      <limit velocity="4.8" effort="1000" lower="${-pi*2.0}" upper="${pi*2.0}" />
+      <limit velocity="4.8" effort="30" lower="${-pi*2.0}" upper="${pi*2.0}" />
       <dynamics damping="0.1" />
     </joint>
@@ -460,5 +460,5 @@
       <child link="left_link_gripper_1"/>
       <axis xyz="1.0 -0.0 -0.0"/>
-      <limit velocity="4.8" effort="1000" lower="${-pi*2.0}" upper="${pi*2.0}" />
+      <limit velocity="4.8" effort="30" lower="${-pi*2.0}" upper="${pi*2.0}" />
       <dynamics damping="0.1" />
     </joint>
@@ -468,5 +468,5 @@
       <child link="neck_link1_1"/>
       <axis xyz="0.0 1.0 -0.0"/>
-      <limit velocity="4.8" effort="1000" lower="${-pi*2.0}" upper="${pi*2.0}" />
+      <limit velocity="4.8" effort="30" lower="${-pi*2.0}" upper="${pi*2.0}" />
       <dynamics damping="0.1" />
     </joint>
@@ -476,5 +476,5 @@
       <child link="neck_link2_1"/>
       <axis xyz="0.0 0.0 1.0"/>
-      <limit velocity="4.8" effort="1000" lower="${-pi*2.0}" upper="${pi*2.0}" />
+      <limit velocity="4.8" effort="30" lower="${-pi*2.0}" upper="${pi*2.0}" />
       <dynamics damping="0.1" />
     </joint>
