Commit message: Add rviz

File: avatar_description/urdf/follower/follower_arm.urdf.xacro (robot description, xacro)
@@ -9,4 +9,5 @@
         <origin xyz="0 0 0" rpy="0 0 0" />
         <geometry>
+          <box size="0.04 0.04 0.02" />
           <!-- <mesh filename="${meshes_file_direction}/follower_01_base.stl" scale="0.001 0.001 0.001" /> -->
         </geometry>
@@ -18,4 +19,5 @@
         <origin xyz="0 0 0" rpy="0 0 0" />
         <geometry>
+          <box size="0.04 0.04 0.02" />
           <!-- <mesh filename="${meshes_file_direction}/follower_01_base.stl" scale="0.001 0.001 0.001" /> -->
         </geometry>
@@ -44,4 +46,5 @@
         <origin xyz="0 0 0" rpy="0 0 0" />
         <geometry>
+          <box size="0.04 0.04 0.02" />
           <!-- <mesh filename="${meshes_file_direction}/follower_02_link1.stl" scale="0.001 0.001 0.001" /> -->
         </geometry>
@@ -53,4 +56,5 @@
         <origin xyz="0 0 0" rpy="0 0 0" />
         <geometry>
+          <box size="0.04 0.04 0.02" />
           <!-- <mesh filename="${meshes_file_direction}/follower_02_link1.stl" scale="0.001 0.001 0.001" /> -->
         </geometry>
@@ -79,4 +83,5 @@
         <origin xyz="0 0 0" rpy="0 0 0" />
         <geometry>
+          <box size="0.04 0.04 0.02" />
           <!-- <mesh filename="${meshes_file_direction}/follower_03_link2.stl" scale="0.001 0.001 0.001" /> -->
         </geometry>
@@ -88,4 +93,5 @@
         <origin xyz="0 0 0" rpy="0 0 0" />
         <geometry>
+          <box size="0.04 0.04 0.02" />
           <!-- <mesh filename="${meshes_file_direction}/follower_03_link2.stl" scale="0.001 0.001 0.001" /> -->
         </geometry>

Commit message: Add urdf debug

File: avatar_description/urdf/follower/follower_arm.urdf.xacro (robot description, xacro)
@@ -7,5 +7,5 @@
     <link name="${prefix}link0" >
       <visual>
-        <origin xyz="0 0 0" rpy="0 0 0" />
+        <origin xyz="0 0 0.01" rpy="0 0 0" />
         <geometry>
           <box size="0.04 0.04 0.02" />
@@ -17,5 +17,5 @@
       </visual>
       <collision>
-        <origin xyz="0 0 0" rpy="0 0 0" />
+        <origin xyz="0 0 0.01" rpy="0 0 0" />
         <geometry>
           <box size="0.04 0.04 0.02" />
@@ -44,7 +44,7 @@
     <link name="${prefix}link1" >
       <visual>
-        <origin xyz="0 0 0" rpy="0 0 0" />
+        <origin xyz="0 0 0.05" rpy="0 0 0" />
         <geometry>
-          <box size="0.04 0.04 0.02" />
+          <box size="0.04 0.04 0.10" />
           <!-- <mesh filename="${meshes_file_direction}/follower_02_link1.stl" scale="0.001 0.001 0.001" /> -->
         </geometry>
@@ -54,7 +54,7 @@
       </visual>
       <collision>
-        <origin xyz="0 0 0" rpy="0 0 0" />
+        <origin xyz="0 0 0.05" rpy="0 0 0" />
         <geometry>
-          <box size="0.04 0.04 0.02" />
+          <box size="0.04 0.04 0.10" />
           <!-- <mesh filename="${meshes_file_direction}/follower_02_link1.stl" scale="0.001 0.001 0.001" /> -->
         </geometry>
@@ -81,7 +81,7 @@
     <link name="${prefix}link2" >
       <visual>
-        <origin xyz="0 0 0" rpy="0 0 0" />
+        <origin xyz="0 0 0.05" rpy="0 0 0" />
         <geometry>
-          <box size="0.04 0.04 0.02" />
+          <box size="0.04 0.04 0.10" />
           <!-- <mesh filename="${meshes_file_direction}/follower_03_link2.stl" scale="0.001 0.001 0.001" /> -->
         </geometry>
@@ -91,7 +91,7 @@
       </visual>
       <collision>
-        <origin xyz="0 0 0" rpy="0 0 0" />
+        <origin xyz="0 0 0.05" rpy="0 0 0" />
         <geometry>
-          <box size="0.04 0.04 0.02" />
+          <box size="0.04 0.04 0.10" />
           <!-- <mesh filename="${meshes_file_direction}/follower_03_link2.stl" scale="0.001 0.001 0.001" /> -->
         </geometry>

Commit message: Add arm Urdf

File: avatar_description/urdf/follower/follower_arm.urdf.xacro (robot description, xacro)
@@ -2,12 +2,17 @@
 <robot xmlns:xacro="http://www.ros.org/wiki/xacro">
   <xacro:macro name="follower" params="prefix">
-    <!-- test -->
-    <!-- <xacro:property name="meshes_file_direction" value="package://avatar_description/meshes/follower/" /> -->
+    <xacro:property name="pi" value="3.1415926535" />
+    <xacro:property name="robot_thickness" value="0.08" />
+    <xacro:property name="body_height" value="0.5" />
+    <xacro:property name="body_width" value="0.4" />
+    <xacro:property name="arm1_height" value="0.15"/>
+    <xacro:property name="arm2_height" value="0.10"/>
+    <xacro:property name="gripper_height" value="0.05"/>
     <!-- link0 -->
     <link name="${prefix}link0" >
       <visual>
-        <origin xyz="0 0 0.01" rpy="0 0 0" />
-        <geometry>
-          <box size="0.04 0.04 0.02" />
+        <origin xyz="0 0 ${body_height/2}" rpy="0 0 0" />
+        <geometry>
+          <box size="${body_width} ${robot_thickness} ${body_height}" />
           <!-- <mesh filename="${meshes_file_direction}/follower_01_base.stl" scale="0.001 0.001 0.001" /> -->
         </geometry>
@@ -17,12 +22,8 @@
       </visual>
       <collision>
-        <origin xyz="0 0 0.01" rpy="0 0 0" />
-        <geometry>
-          <box size="0.04 0.04 0.02" />
-          <!-- <mesh filename="${meshes_file_direction}/follower_01_base.stl" scale="0.001 0.001 0.001" /> -->
-        </geometry>
-        <material name="grey">
-          <color rgba="0.2 0.2 0.2 1" />
-        </material>
+        <origin xyz="0 0 ${body_height/2}" rpy="0 0 0" />
+        <geometry>
+          <box size="${body_width} ${robot_thickness} ${body_height}" />
+        </geometry>
       </collision>
       <inertial>
@@ -33,33 +34,28 @@
     </link>
     <!-- joint1 -->
-    <joint name="${prefix}joint1" type="revolute">
+    <joint name="${prefix}right_joint1" type="revolute">
       <parent link="${prefix}link0" />
-      <child link="${prefix}link1" />
-      <origin xyz="0 0 0.02" rpy="0 0 0" />
-      <axis xyz="0 0 1" />
-      <limit velocity="4.8" effort="1000" lower="${-pi*2.0}" upper="${pi*2.0}" />
+      <child link="${prefix}right_link1" />
+      <origin xyz="${body_width/2} 0 ${body_height - robot_thickness/2}" rpy="0 0 0" />
+      <axis xyz="1 0 0" />
+      <limit velocity="4.8" effort="1000" lower="${-pi}" upper="${pi}" />
       <dynamics damping="0.05" />
     </joint>
     <!-- link1 -->
-    <link name="${prefix}link1" >
-      <visual>
-        <origin xyz="0 0 0.05" rpy="0 0 0" />
-        <geometry>
-          <box size="0.04 0.04 0.10" />
-          <!-- <mesh filename="${meshes_file_direction}/follower_02_link1.stl" scale="0.001 0.001 0.001" /> -->
-        </geometry>
-        <material name="grey">
-          <color rgba="0.2 0.2 0.2 1" />
-        </material>
-      </visual>
-      <collision>
-        <origin xyz="0 0 0.05" rpy="0 0 0" />
-        <geometry>
-          <box size="0.04 0.04 0.10" />
-          <!-- <mesh filename="${meshes_file_direction}/follower_02_link1.stl" scale="0.001 0.001 0.001" /> -->
-        </geometry>
-        <material name="grey">
-          <color rgba="0.2 0.2 0.2 1" />
-        </material>
+    <link name="${prefix}right_link1" >
+      <visual>
+        <origin xyz="${robot_thickness/2} 0 0" rpy="${pi/2} 0 0" />
+        <geometry>
+          <cylinder radius="${robot_thickness/2}" length="${robot_thickness}"/>
+        </geometry>
+        <material name="grey">
+          <color rgba="0.2 0.2 0.2 1" />
+        </material>
+      </visual>
+      <collision>
+        <origin xyz="${robot_thickness/2} 0 0" rpy="${pi/2} 0 0" />
+        <geometry>
+          <cylinder radius="${robot_thickness/2}" length="${robot_thickness}"/>
+        </geometry>
       </collision>
       <inertial>
@@ -70,33 +66,28 @@
     </link>
     <!-- joint2 -->
-    <joint name="${prefix}joint2" type="revolute">
-      <parent link="${prefix}link1" />
-      <child link="${prefix}link2" />
-      <origin xyz="0 0 0.10" rpy="0 0 0" />
+    <joint name="${prefix}right_joint2" type="revolute">
+      <parent link="${prefix}right_link1" />
+      <child link="${prefix}right_link2" />
+      <origin xyz="${robot_thickness/2} 0 0" rpy="0 0 0" />
       <axis xyz="0 1 0" />
-      <limit velocity="4.8" effort="1000" lower="${-pi*2.0}" upper="${pi*2.0}" />
+      <limit velocity="4.8" effort="1000" lower="${-pi}" upper="${pi/2}" />
       <dynamics damping="0.1" />
     </joint>
     <!-- link2 -->
-    <link name="${prefix}link2" >
-      <visual>
-        <origin xyz="0 0 0.05" rpy="0 0 0" />
-        <geometry>
-          <box size="0.04 0.04 0.10" />
-          <!-- <mesh filename="${meshes_file_direction}/follower_03_link2.stl" scale="0.001 0.001 0.001" /> -->
-        </geometry>
-        <material name="grey">
-          <color rgba="0.2 0.2 0.2 1" />
-        </material>
-      </visual>
-      <collision>
-        <origin xyz="0 0 0.05" rpy="0 0 0" />
-        <geometry>
-          <box size="0.04 0.04 0.10" />
-          <!-- <mesh filename="${meshes_file_direction}/follower_03_link2.stl" scale="0.001 0.001 0.001" /> -->
-        </geometry>
-        <material name="grey">
-          <color rgba="0.2 0.2 0.2 1" />
-        </material>
+    <link name="${prefix}right_link2" >
+      <visual>
+        <origin xyz="0 0 ${-robot_thickness/2 - arm1_height/2}" rpy="0 0 0" />
+        <geometry>
+          <box size="${robot_thickness} ${robot_thickness} ${arm1_height}" />
+        </geometry>
+        <material name="grey">
+          <color rgba="0.2 0.2 0.2 1" />
+        </material>
+      </visual>
+      <collision>
+        <origin xyz="0 0 ${-robot_thickness/2 - arm1_height/2}" rpy="0 0 0" />
+        <geometry>
+          <box size="${robot_thickness} ${robot_thickness} ${arm1_height}" />
+        </geometry>
       </collision>
       <inertial>
@@ -106,4 +97,132 @@
       </inertial>
     </link>
+    <!-- joint3 -->
+    <joint name="${prefix}right_joint3" type="revolute">
+      <parent link="${prefix}right_link2" />
+      <child link="${prefix}right_link3" />
+      <origin xyz="0 0 ${-arm1_height - robot_thickness/2}" rpy="0 0 0" />
+      <axis xyz="0 0 -1" />
+      <limit velocity="4.8" effort="1000" lower="${-pi/2}" upper="${pi/2}" />
+      <dynamics damping="0.1" />
+    </joint>
+    <!-- link3 -->
+    <link name="${prefix}right_link3" >
+      <visual>
+        <origin xyz="0 0 ${-robot_thickness/2}" rpy="${pi/2} 0 ${pi/2}" />
+        <geometry>
+          <cylinder radius="${robot_thickness/2}" length="${robot_thickness}"/>
+        </geometry>
+        <material name="grey">
+          <color rgba="0.2 0.2 0.2 1" />
+        </material>
+      </visual>
+      <collision>
+        <origin xyz="${robot_thickness/2} 0 0" rpy="${pi/2} 0 0" />
+        <geometry>
+          <cylinder radius="${robot_thickness/2}" length="${robot_thickness}"/>
+        </geometry>
+      </collision>
+      <inertial>
+        <origin xyz="0 0 0.05" />
+        <mass value="1.0e-1" />
+        <inertia ixx="5e-5" ixy="0" ixz="0" iyy="5e-5" iyz="0" izz="1e-5" />
+      </inertial>
+    </link>
+    <!-- joint4 -->
+    <joint name="${prefix}right_joint4" type="revolute">
+      <parent link="${prefix}right_link3" />
+      <child link="${prefix}right_link4" />
+      <origin xyz="0 0 ${-robot_thickness/2}" rpy="0 0 0" />
+      <axis xyz="1 0 0" />
+      <limit velocity="4.8" effort="1000" lower="0" upper="${pi}" />
+      <dynamics damping="0.1" />
+    </joint>
+    <!-- link4 -->
+    <link name="${prefix}right_link4" >
+      <visual>
+        <origin xyz="0 0 ${-robot_thickness/2 - arm2_height/2}" rpy="0 0 0" />
+        <geometry>
+          <box size="${robot_thickness} ${robot_thickness} ${arm2_height}" />
+        </geometry>
+        <material name="grey">
+          <color rgba="0.2 0.2 0.2 1" />
+        </material>
+      </visual>
+      <collision>
+        <origin xyz="0 0 ${-robot_thickness/2 - arm2_height/2}" rpy="0 0 0" />
+        <geometry>
+          <box size="${robot_thickness} ${robot_thickness} ${arm2_height}" />
+        </geometry>
+      </collision>
+      <inertial>
+        <origin xyz="0 0 0.05" />
+        <mass value="8.0e-2" />
+        <inertia ixx="4e-5" ixy="0" ixz="0" iyy="4e-5" iyz="0" izz="8e-6" />
+      </inertial>
+    </link>
+     <!-- joint5 -->
+    <joint name="${prefix}right_joint5" type="revolute">
+      <parent link="${prefix}right_link4" />
+      <child link="${prefix}right_link5" />
+      <origin xyz="0 0 ${-arm2_height - robot_thickness/2}" rpy="0 0 0" />
+      <axis xyz="0 0 -1" />
+      <limit velocity="4.8" effort="1000" lower="${-pi/2}" upper="${pi/2}" />
+      <dynamics damping="0.1" />
+    </joint>
+    <!-- link5 -->
+    <link name="${prefix}right_link5" >
+      <visual>
+        <origin xyz="0 0 ${-robot_thickness/2}" rpy="${pi/2} 0 ${pi/2}" />
+        <geometry>
+          <cylinder radius="${robot_thickness/2}" length="${robot_thickness}"/>
+        </geometry>
+        <material name="grey">
+          <color rgba="0.2 0.2 0.2 1" />
+        </material>
+      </visual>
+      <collision>
+        <origin xyz="${robot_thickness/2} 0 0" rpy="${pi/2} 0 0" />
+        <geometry>
+          <cylinder radius="${robot_thickness/2}" length="${robot_thickness}"/>
+        </geometry>
+      </collision>
+      <inertial>
+        <origin xyz="0 0 0.05" />
+        <mass value="1.0e-1" />
+        <inertia ixx="5e-5" ixy="0" ixz="0" iyy="5e-5" iyz="0" izz="1e-5" />
+      </inertial>
+    </link>
+    <!-- joint6 -->
+    <joint name="${prefix}right_joint6" type="revolute">
+      <parent link="${prefix}right_link5" />
+      <child link="${prefix}right_link6" />
+      <origin xyz="0 0 ${-robot_thickness/2}" rpy="0 0 0" />
+      <axis xyz="1 0 0" />
+      <limit velocity="4.8" effort="1000" lower="${-pi/2}" upper="${pi/2}" />
+      <dynamics damping="0.1" />
+    </joint>
+    <!-- link6 -->
+    <link name="${prefix}right_link6" >
+      <visual>
+        <origin xyz="0 0 ${-robot_thickness/2 - gripper_height/2}" rpy="0 0 0" />
+        <geometry>
+          <box size="${robot_thickness} ${robot_thickness} ${gripper_height}" />
+        </geometry>
+        <material name="grey">
+          <color rgba="0.2 0.2 0.2 1" />
+        </material>
+      </visual>
+      <collision>
+        <origin xyz="0 0 ${-robot_thickness/2 - gripper_height/2}" rpy="0 0 0" />
+        <geometry>
+          <box size="${robot_thickness} ${robot_thickness} ${gripper_height}" />
+        </geometry>
+      </collision>
+      <inertial>
+        <origin xyz="0 0 0.05" />
+        <mass value="8.0e-2" />
+        <inertia ixx="4e-5" ixy="0" ixz="0" iyy="4e-5" iyz="0" izz="8e-6" />
+      </inertial>
+    </link>
   </xacro:macro>
 </robot>

Commit message: Edit joint

File: avatar_description/urdf/follower/follower_arm.urdf.xacro (robot description, xacro)
@@ -265,5 +265,5 @@
       <origin xyz="${-robot_thickness/2} 0 0" rpy="0 0 0" />
       <axis xyz="0 1 0" />
-      <limit velocity="4.8" effort="1000" lower="${-pi/2}" upper="${-pi}" />
+      <limit velocity="4.8" effort="1000" lower="${-pi/2}" upper="${pi}" />
       <dynamics damping="0.1" />
     </joint>
