Commit message: Edit 경로

File: avatar_description/urdf/follower/follower_arm.urdf.xacro (robot description, xacro)
@@ -20,5 +20,5 @@
         <origin xyz="0 0 0" rpy="0 0 0"/>
         <geometry>
-          <mesh filename="package://avatar_description/meshes/follower/base_link.stl" scale="0.01 0.01 0.01"/>
+          <mesh filename="file://$(find avatar_description)/meshes/follower/base_link.stl" scale="0.01 0.01 0.01"/>
         </geometry>
         <material name="dark_gray"/>
@@ -27,5 +27,5 @@
         <origin xyz="0 0 0" rpy="0 0 0"/>
         <geometry>
-          <mesh filename="package://avatar_description/meshes/follower/base_link.stl" scale="0.01 0.01 0.01"/>
+          <mesh filename="file://$(find avatar_description)/meshes/follower/base_link.stl" scale="0.01 0.01 0.01"/>
         </geometry>
       </collision>
@@ -40,5 +40,5 @@
         <origin xyz="0.00025 -0.1025 -0.6155" rpy="0 0 0"/>
         <geometry>
-          <mesh filename="package://avatar_description/meshes/follower/left_link1_1.stl" scale="0.01 0.01 0.01"/>
+          <mesh filename="file://$(find avatar_description)/meshes/follower/left_link1_1.stl" scale="0.01 0.01 0.01"/>
         </geometry>
         <material name="dark_gray"/>
@@ -47,5 +47,5 @@
         <origin xyz="0.00025 -0.1025 -0.6155" rpy="0 0 0"/>
         <geometry>
-          <mesh filename="package://avatar_description/meshes/follower/left_link1_1.stl" scale="0.01 0.01 0.01"/>
+          <mesh filename="file://$(find avatar_description)/meshes/follower/left_link1_1.stl" scale="0.01 0.01 0.01"/>
         </geometry>
       </collision>
@@ -60,5 +60,5 @@
         <origin xyz="-0.00025 0.1025 -0.6155" rpy="0 0 0"/>
         <geometry>
-          <mesh filename="package://avatar_description/meshes/follower/right_link1_1.stl" scale="0.01 0.01 0.01"/>
+          <mesh filename="file://$(find avatar_description)/meshes/follower/right_link1_1.stl" scale="0.01 0.01 0.01"/>
         </geometry>
         <material name="dark_gray"/>
@@ -67,5 +67,5 @@
         <origin xyz="-0.00025 0.1025 -0.6155" rpy="0 0 0"/>
         <geometry>
-          <mesh filename="package://avatar_description/meshes/follower/right_link1_1.stl" scale="0.01 0.01 0.01"/>
+          <mesh filename="file://$(find avatar_description)/meshes/follower/right_link1_1.stl" scale="0.01 0.01 0.01"/>
         </geometry>
       </collision>
@@ -80,5 +80,5 @@
         <origin xyz="-0.00025 -0.0194 -0.6478" rpy="0 0 0"/>
         <geometry>
-          <mesh filename="package://avatar_description/meshes/follower/neck_link1_1.stl" scale="0.01 0.01 0.01"/>
+          <mesh filename="file://$(find avatar_description)/meshes/follower/neck_link1_1.stl" scale="0.01 0.01 0.01"/>
         </geometry>
         <material name="dark_gray"/>
@@ -87,5 +87,5 @@
         <origin xyz="-0.00025 -0.0194 -0.6478" rpy="0 0 0"/>
         <geometry>
-          <mesh filename="package://avatar_description/meshes/follower/neck_link1_1.stl" scale="0.01 0.01 0.01"/>
+          <mesh filename="file://$(find avatar_description)/meshes/follower/neck_link1_1.stl" scale="0.01 0.01 0.01"/>
         </geometry>
       </collision>
@@ -100,5 +100,5 @@
         <origin xyz="-0.00025 -0.0004 -0.70755" rpy="0 0 0"/>
         <geometry>
-          <mesh filename="package://avatar_description/meshes/follower/neck_link2_1.stl" scale="0.01 0.01 0.01"/>
+          <mesh filename="file://$(find avatar_description)/meshes/follower/neck_link2_1.stl" scale="0.01 0.01 0.01"/>
         </geometry>
         <material name="white"/>
@@ -107,5 +107,5 @@
         <origin xyz="-0.00025 -0.0004 -0.70755" rpy="0 0 0"/>
         <geometry>
-          <mesh filename="package://avatar_description/meshes/follower/neck_link2_1.stl" scale="0.01 0.01 0.01"/>
+          <mesh filename="file://$(find avatar_description)/meshes/follower/neck_link2_1.stl" scale="0.01 0.01 0.01"/>
         </geometry>
       </collision>
@@ -120,5 +120,5 @@
         <origin xyz="-0.02425 -0.1525 -0.6155" rpy="0 0 0"/>
         <geometry>
-          <mesh filename="package://avatar_description/meshes/follower/left_link2_1.stl" scale="0.01 0.01 0.01"/>
+          <mesh filename="file://$(find avatar_description)/meshes/follower/left_link2_1.stl" scale="0.01 0.01 0.01"/>
         </geometry>
         <material name="dark_gray"/>
@@ -127,5 +127,5 @@
         <origin xyz="-0.02425 -0.1525 -0.6155" rpy="0 0 0"/>
         <geometry>
-          <mesh filename="package://avatar_description/meshes/follower/left_link2_1.stl" scale="0.01 0.01 0.01"/>
+          <mesh filename="file://$(find avatar_description)/meshes/follower/left_link2_1.stl" scale="0.01 0.01 0.01"/>
         </geometry>
       </collision>
@@ -140,5 +140,5 @@
         <origin xyz="0.00025 -0.1525 -0.45775" rpy="0 0 0"/>
         <geometry>
-          <mesh filename="package://avatar_description/meshes/follower/left_link3_1.stl" scale="0.01 0.01 0.01"/>
+          <mesh filename="file://$(find avatar_description)/meshes/follower/left_link3_1.stl" scale="0.01 0.01 0.01"/>
         </geometry>
         <material name="dark_gray"/>
@@ -147,5 +147,5 @@
         <origin xyz="0.00025 -0.1525 -0.45775" rpy="0 0 0"/>
         <geometry>
-          <mesh filename="package://avatar_description/meshes/follower/left_link3_1.stl" scale="0.01 0.01 0.01"/>
+          <mesh filename="file://$(find avatar_description)/meshes/follower/left_link3_1.stl" scale="0.01 0.01 0.01"/>
         </geometry>
       </collision>
@@ -160,5 +160,5 @@
         <origin xyz="0.00025 -0.1715 -0.42625" rpy="0 0 0"/>
         <geometry>
-          <mesh filename="package://avatar_description/meshes/follower/left_link4_1.stl" scale="0.01 0.01 0.01"/>
+          <mesh filename="file://$(find avatar_description)/meshes/follower/left_link4_1.stl" scale="0.01 0.01 0.01"/>
         </geometry>
         <material name="dark_gray"/>
@@ -167,5 +167,5 @@
         <origin xyz="0.00025 -0.1715 -0.42625" rpy="0 0 0"/>
         <geometry>
-          <mesh filename="package://avatar_description/meshes/follower/left_link4_1.stl" scale="0.01 0.01 0.01"/>
+          <mesh filename="file://$(find avatar_description)/meshes/follower/left_link4_1.stl" scale="0.01 0.01 0.01"/>
         </geometry>
       </collision>
@@ -180,5 +180,5 @@
         <origin xyz="0.00025 -0.1525 -0.28615" rpy="0 0 0"/>
         <geometry>
-          <mesh filename="package://avatar_description/meshes/follower/left_link5_1.stl" scale="0.01 0.01 0.01"/>
+          <mesh filename="file://$(find avatar_description)/meshes/follower/left_link5_1.stl" scale="0.01 0.01 0.01"/>
         </geometry>
         <material name="dark_gray"/>
@@ -187,5 +187,5 @@
         <origin xyz="0.00025 -0.1525 -0.28615" rpy="0 0 0"/>
         <geometry>
-          <mesh filename="package://avatar_description/meshes/follower/left_link5_1.stl" scale="0.01 0.01 0.01"/>
+          <mesh filename="file://$(find avatar_description)/meshes/follower/left_link5_1.stl" scale="0.01 0.01 0.01"/>
         </geometry>
       </collision>
@@ -200,5 +200,5 @@
         <origin xyz="0.00025 -0.1715 -0.25465" rpy="0 0 0"/>
         <geometry>
-          <mesh filename="package://avatar_description/meshes/follower/left_link6_1.stl" scale="0.01 0.01 0.01"/>
+          <mesh filename="file://$(find avatar_description)/meshes/follower/left_link6_1.stl" scale="0.01 0.01 0.01"/>
         </geometry>
         <material name="dark_gray"/>
@@ -207,5 +207,5 @@
         <origin xyz="0.00025 -0.1715 -0.25465" rpy="0 0 0"/>
         <geometry>
-          <mesh filename="package://avatar_description/meshes/follower/left_link6_1.stl" scale="0.01 0.01 0.01"/>
+          <mesh filename="file://$(find avatar_description)/meshes/follower/left_link6_1.stl" scale="0.01 0.01 0.01"/>
         </geometry>
       </collision>
@@ -220,5 +220,5 @@
         <origin xyz="-0.01875 -0.1629 -0.20515" rpy="0 0 0"/>
         <geometry>
-          <mesh filename="package://avatar_description/meshes/follower/left_link_gripper_1.stl" scale="0.01 0.01 0.01"/>
+          <mesh filename="file://$(find avatar_description)/meshes/follower/left_link_gripper_1.stl" scale="0.01 0.01 0.01"/>
         </geometry>
         <material name="dark_gray"/>
@@ -227,5 +227,5 @@
         <origin xyz="-0.01875 -0.1629 -0.20515" rpy="0 0 0"/>
         <geometry>
-          <mesh filename="package://avatar_description/meshes/follower/left_link_gripper_1.stl" scale="0.01 0.01 0.01"/>
+          <mesh filename="file://$(find avatar_description)/meshes/follower/left_link_gripper_1.stl" scale="0.01 0.01 0.01"/>
         </geometry>
       </collision>
@@ -240,5 +240,5 @@
         <origin xyz="-0.02475 0.1525 -0.6155" rpy="0 0 0"/>
         <geometry>
-          <mesh filename="package://avatar_description/meshes/follower/right_link2_1.stl" scale="0.01 0.01 0.01"/>
+          <mesh filename="file://$(find avatar_description)/meshes/follower/right_link2_1.stl" scale="0.01 0.01 0.01"/>
         </geometry>
         <material name="dark_gray"/>
@@ -247,5 +247,5 @@
         <origin xyz="-0.02475 0.1525 -0.6155" rpy="0 0 0"/>
         <geometry>
-          <mesh filename="package://avatar_description/meshes/follower/right_link2_1.stl" scale="0.01 0.01 0.01"/>
+          <mesh filename="file://$(find avatar_description)/meshes/follower/right_link2_1.stl" scale="0.01 0.01 0.01"/>
         </geometry>
       </collision>
@@ -260,5 +260,5 @@
         <origin xyz="-0.00025 0.1525 -0.45775" rpy="0 0 0"/>
         <geometry>
-          <mesh filename="package://avatar_description/meshes/follower/right_link3_1.stl" scale="0.01 0.01 0.01"/>
+          <mesh filename="file://$(find avatar_description)/meshes/follower/right_link3_1.stl" scale="0.01 0.01 0.01"/>
         </geometry>
         <material name="dark_gray"/>
@@ -267,5 +267,5 @@
         <origin xyz="-0.00025 0.1525 -0.45775" rpy="0 0 0"/>
         <geometry>
-          <mesh filename="package://avatar_description/meshes/follower/right_link3_1.stl" scale="0.01 0.01 0.01"/>
+          <mesh filename="file://$(find avatar_description)/meshes/follower/right_link3_1.stl" scale="0.01 0.01 0.01"/>
         </geometry>
       </collision>
@@ -280,5 +280,5 @@
         <origin xyz="-0.00025 0.1715 -0.42625" rpy="0 0 0"/>
         <geometry>
-          <mesh filename="package://avatar_description/meshes/follower/right_link4_1.stl" scale="0.01 0.01 0.01"/>
+          <mesh filename="file://$(find avatar_description)/meshes/follower/right_link4_1.stl" scale="0.01 0.01 0.01"/>
         </geometry>
         <material name="dark_gray"/>
@@ -287,5 +287,5 @@
         <origin xyz="-0.00025 0.1715 -0.42625" rpy="0 0 0"/>
         <geometry>
-          <mesh filename="package://avatar_description/meshes/follower/right_link4_1.stl" scale="0.01 0.01 0.01"/>
+          <mesh filename="file://$(find avatar_description)/meshes/follower/right_link4_1.stl" scale="0.01 0.01 0.01"/>
         </geometry>
       </collision>
@@ -300,5 +300,5 @@
         <origin xyz="-0.00025 0.1525 -0.28615" rpy="0 0 0"/>
         <geometry>
-          <mesh filename="package://avatar_description/meshes/follower/right_link5_1.stl" scale="0.01 0.01 0.01"/>
+          <mesh filename="file://$(find avatar_description)/meshes/follower/right_link5_1.stl" scale="0.01 0.01 0.01"/>
         </geometry>
         <material name="dark_gray"/>
@@ -307,5 +307,5 @@
         <origin xyz="-0.00025 0.1525 -0.28615" rpy="0 0 0"/>
         <geometry>
-          <mesh filename="package://avatar_description/meshes/follower/right_link5_1.stl" scale="0.01 0.01 0.01"/>
+          <mesh filename="file://$(find avatar_description)/meshes/follower/right_link5_1.stl" scale="0.01 0.01 0.01"/>
         </geometry>
       </collision>
@@ -320,5 +320,5 @@
         <origin xyz="-0.00025 0.1715 -0.25465" rpy="0 0 0"/>
         <geometry>
-          <mesh filename="package://avatar_description/meshes/follower/right_link6_1.stl" scale="0.01 0.01 0.01"/>
+          <mesh filename="file://$(find avatar_description)/meshes/follower/right_link6_1.stl" scale="0.01 0.01 0.01"/>
         </geometry>
         <material name="dark_gray"/>
@@ -327,5 +327,5 @@
         <origin xyz="-0.00025 0.1715 -0.25465" rpy="0 0 0"/>
         <geometry>
-          <mesh filename="package://avatar_description/meshes/follower/right_link6_1.stl" scale="0.01 0.01 0.01"/>
+          <mesh filename="file://$(find avatar_description)/meshes/follower/right_link6_1.stl" scale="0.01 0.01 0.01"/>
         </geometry>
       </collision>
@@ -340,5 +340,5 @@
         <origin xyz="-0.01925 0.1645 -0.20515" rpy="0 0 0"/>
         <geometry>
-          <mesh filename="package://avatar_description/meshes/follower/right_link_gripper_1.stl" scale="0.01 0.01 0.01"/>
+          <mesh filename="file://$(find avatar_description)/meshes/follower/right_link_gripper_1.stl" scale="0.01 0.01 0.01"/>
         </geometry>
         <material name="dark_gray"/>
@@ -347,5 +347,5 @@
         <origin xyz="-0.01925 0.1645 -0.20515" rpy="0 0 0"/>
         <geometry>
-          <mesh filename="package://avatar_description/meshes/follower/right_link_gripper_1.stl" scale="0.01 0.01 0.01"/>
+          <mesh filename="file://$(find avatar_description)/meshes/follower/right_link_gripper_1.stl" scale="0.01 0.01 0.01"/>
         </geometry>
       </collision>

Commit message: Add joint effort

File: avatar_description/urdf/follower/follower_arm.urdf.xacro (robot description, xacro)
@@ -356,4 +356,6 @@
       <child link="right_link1_1"/>
       <axis xyz="-0.0 -1.0 0.0"/>
+      <limit velocity="4.8" effort="1000" lower="${-pi*2.0}" upper="${pi*2.0}" />
+      <dynamics damping="0.1" />
     </joint>
     <joint name="right_joint2" type="continuous">
@@ -362,4 +364,6 @@
       <child link="right_link2_1"/>
       <axis xyz="-1.0 -0.0 0.0"/>
+      <limit velocity="4.8" effort="1000" lower="${-pi*2.0}" upper="${pi*2.0}" />
+      <dynamics damping="0.1" />
     </joint>
     <joint name="right_joint3" type="continuous">
@@ -368,10 +372,14 @@
       <child link="right_link3_1"/>
       <axis xyz="0.0 -0.0 -1.0"/>
+      <limit velocity="4.8" effort="1000" lower="${-pi*2.0}" upper="${pi*2.0}" />
+      <dynamics damping="0.1" />
     </joint>
     <joint name="right_joint4" type="continuous">
       <origin xyz="0.0 -0.019 -0.0315" rpy="0 0 0"/>
       <parent link="right_link3_1"/>
-      <child link="right_link4_1"/>p
+      <child link="right_link4_1"/>
       <axis xyz="0.0 1.0 -0.0"/>
+      <limit velocity="4.8" effort="1000" lower="${-pi*2.0}" upper="${pi*2.0}" />
+      <dynamics damping="0.1" />
     </joint>
     <joint name="right_joint5" type="continuous">
@@ -380,4 +388,6 @@
       <child link="right_link5_1"/>
       <axis xyz="0.0 0.0 -1.0"/>
+      <limit velocity="4.8" effort="1000" lower="${-pi*2.0}" upper="${pi*2.0}" />
+      <dynamics damping="0.1" />
     </joint>
     <joint name="right_joint6" type="continuous">
@@ -386,4 +396,6 @@
       <child link="right_link6_1"/>
       <axis xyz="0.0 1.0 0.0"/>
+      <limit velocity="4.8" effort="1000" lower="${-pi*2.0}" upper="${pi*2.0}" />
+      <dynamics damping="0.1" />
     </joint>
     <joint name="right_joint_gripper" type="continuous">
@@ -392,4 +404,6 @@
       <child link="right_link_gripper_1"/>
       <axis xyz="1.0 -0.0 -0.0"/>
+      <limit velocity="4.8" effort="1000" lower="${-pi*2.0}" upper="${pi*2.0}" />
+      <dynamics damping="0.1" />
     </joint>
     <joint name="left_joint1" type="continuous">
@@ -398,4 +412,6 @@
       <child link="left_link1_1"/>
       <axis xyz="0.0 1.0 0.0"/>
+      <limit velocity="4.8" effort="1000" lower="${-pi*2.0}" upper="${pi*2.0}" />
+      <dynamics damping="0.1" />
     </joint>
     <joint name="left_joint2" type="continuous">
@@ -404,4 +420,6 @@
       <child link="left_link2_1"/>
       <axis xyz="-1.0 -0.0 -0.0"/>
+      <limit velocity="4.8" effort="1000" lower="${-pi*2.0}" upper="${pi*2.0}" />
+      <dynamics damping="0.1" />
     </joint>
     <joint name="left_joint3" type="continuous">
@@ -410,4 +428,6 @@
       <child link="left_link3_1"/>
       <axis xyz="0.0 -0.0 -1.0"/>
+      <limit velocity="4.8" effort="1000" lower="${-pi*2.0}" upper="${pi*2.0}" />
+      <dynamics damping="0.1" />
     </joint>
     <joint name="left_joint4" type="continuous">
@@ -416,4 +436,6 @@
       <child link="left_link4_1"/>
       <axis xyz="-0.0 -1.0 0.0"/>
+      <limit velocity="4.8" effort="1000" lower="${-pi*2.0}" upper="${pi*2.0}" />
+      <dynamics damping="0.1" />
     </joint>
     <joint name="left_joint5" type="continuous">
@@ -422,4 +444,6 @@
       <child link="left_link5_1"/>
       <axis xyz="0.0 0.0 -1.0"/>
+      <limit velocity="4.8" effort="1000" lower="${-pi*2.0}" upper="${pi*2.0}" />
+      <dynamics damping="0.1" />
     </joint>
     <joint name="left_joint6" type="continuous">
@@ -428,4 +452,6 @@
       <child link="left_link6_1"/>
       <axis xyz="-0.0 -1.0 -0.0"/>
+      <limit velocity="4.8" effort="1000" lower="${-pi*2.0}" upper="${pi*2.0}" />
+      <dynamics damping="0.1" />
     </joint>
     <joint name="left_joint_gripper" type="continuous">
@@ -434,4 +460,6 @@
       <child link="left_link_gripper_1"/>
       <axis xyz="1.0 -0.0 -0.0"/>
+      <limit velocity="4.8" effort="1000" lower="${-pi*2.0}" upper="${pi*2.0}" />
+      <dynamics damping="0.1" />
     </joint>
     <joint name="neck_joint1" type="continuous">
@@ -440,4 +468,6 @@
       <child link="neck_link1_1"/>
       <axis xyz="0.0 1.0 -0.0"/>
+      <limit velocity="4.8" effort="1000" lower="${-pi*2.0}" upper="${pi*2.0}" />
+      <dynamics damping="0.1" />
     </joint>
     <joint name="neck_joint2" type="continuous">
@@ -446,4 +476,6 @@
       <child link="neck_link2_1"/>
       <axis xyz="0.0 0.0 1.0"/>
+      <limit velocity="4.8" effort="1000" lower="${-pi*2.0}" upper="${pi*2.0}" />
+      <dynamics damping="0.1" />
     </joint>
   </xacro:macro>

Commit message: 충돌 추가 시도 2

File: avatar_description/urdf/follower/follower_arm.urdf.xacro (robot description, xacro)
@@ -479,4 +479,30 @@
       <dynamics damping="0.1" />
     </joint>
+    <gazebo reference="left_link_gripper_1">
+      <self_collide>true</self_collide>
+      <sensor name="left_gripper_bumper" type="contact">
+        <always_on>true</always_on>
+        <update_rate>50.0</update_rate>
+        <contact>
+          <collision>left_link_gripper_1_collision</collision>
+        </contact>
+      </sensor>
+    </gazebo>
+    <gazebo reference="right_link_gripper_1">
+      <self_collide>true</self_collide>
+      <sensor name="right_gripper_bumper" type="contact">
+        <always_on>true</always_on>
+        <update_rate>50.0</update_rate>
+        <contact>
+          <collision>right_link_gripper_1_collision</collision>
+        </contact>
+      </sensor>
+    </gazebo>
+    <gazebo reference="left_link6_1"><self_collide>true</self_collide></gazebo>
+    <gazebo reference="left_link5_1"><self_collide>true</self_collide></gazebo>
+    <gazebo reference="left_link4_1"><self_collide>true</self_collide></gazebo>
+    <gazebo reference="right_link6_1"><self_collide>true</self_collide></gazebo>
+    <gazebo reference="right_link5_1"><self_collide>true</self_collide></gazebo>
+    <gazebo reference="right_link4_1"><self_collide>true</self_collide></gazebo>
   </xacro:macro>
 </robot>

Commit message: 3try to chungdol

File: avatar_description/urdf/follower/follower_arm.urdf.xacro (robot description, xacro)
@@ -224,5 +224,5 @@
         <material name="dark_gray"/>
       </visual>
-      <collision>
+      <collision name="${prefix}left_link_gripper_1_collision">
         <origin xyz="-0.01875 -0.1629 -0.20515" rpy="0 0 0"/>
         <geometry>
@@ -344,5 +344,5 @@
         <material name="dark_gray"/>
       </visual>
-      <collision>
+      <collision name="${prefix}right_link_gripper_1_collision">
         <origin xyz="-0.01925 0.1645 -0.20515" rpy="0 0 0"/>
         <geometry>
@@ -479,4 +479,28 @@
       <dynamics damping="0.1" />
     </joint>
+    <gazebo reference="left_link_gripper_1">
+      <sensor name="left_gripper_bumper" type="contact">
+        <always_on>true</always_on>
+        <update_rate>50.0</update_rate>
+        <contact>
+          <collision>${prefix}left_link_gripper_1_collision_collision</collision>
+        </contact>
+        <plugin filename="libignition-gazebo-contact-system.so"
+                name="ignition::gazebo::systems::Contact">
+        </plugin>
+      </sensor>
+    </gazebo>
+    <gazebo reference="right_link_gripper_1">
+      <sensor name="right_gripper_bumper" type="contact">
+        <always_on>true</always_on>
+        <update_rate>50.0</update_rate>
+        <contact>
+          <collision>${prefix}right_link_gripper_1_collision_collision</collision>
+        </contact>
+        <plugin filename="libignition-gazebo-contact-system.so"
+                name="ignition::gazebo::systems::Contact">
+        </plugin>
+      </sensor>
+    </gazebo>
   </xacro:macro>
 </robot>
