Commit message: urdf 조인트 방향 (실제 로봇과 같게)

File: avatar_description/urdf/follower/follower_arm.urdf.xacro (robot description, xacro)
@@ -355,6 +355,6 @@
       <parent link="base_link"/>
       <child link="right_link1_1"/>
-      <axis xyz="-0.0 -1.0 0.0"/>
-      <limit velocity="4.8" effort="30" lower="${-pi*2.0}" upper="${pi*2.0}" />
+      <axis xyz="0.0 -1.0 0.0"/>
+      <limit velocity="4.8" effort="30" lower="${-pi*0.5}" upper="${pi*0.5}" />
       <dynamics damping="0.1" />
     </joint>
@@ -363,6 +363,6 @@
       <parent link="right_link1_1"/>
       <child link="right_link2_1"/>
-      <axis xyz="-1.0 -0.0 0.0"/>
-      <limit velocity="4.8" effort="30" lower="${-pi*2.0}" upper="${pi*2.0}" />
+      <axis xyz="-1.0 0.0 0.0"/>
+      <limit velocity="4.8" effort="30" lower="${-pi*0.5}" upper="${pi*0.5}" />
       <dynamics damping="0.1" />
     </joint>
@@ -371,6 +371,6 @@
       <parent link="right_link2_1"/>
       <child link="right_link3_1"/>
-      <axis xyz="0.0 -0.0 -1.0"/>
-      <limit velocity="4.8" effort="30" lower="${-pi*2.0}" upper="${pi*2.0}" />
+      <axis xyz="0.0 0.0 -1.0"/>
+      <limit velocity="4.8" effort="30" lower="${-pi*0.5}" upper="${pi*0.5}" />
       <dynamics damping="0.1" />
     </joint>
@@ -379,6 +379,6 @@
       <parent link="right_link3_1"/>
       <child link="right_link4_1"/>
-      <axis xyz="0.0 1.0 -0.0"/>
-      <limit velocity="4.8" effort="30" lower="${-pi*2.0}" upper="${pi*2.0}" />
+      <axis xyz="0.0 -1.0 0.0"/>
+      <limit velocity="4.8" effort="30" lower="${-pi*0.5}" upper="${pi*0.5}" />
       <dynamics damping="0.1" />
     </joint>
@@ -388,5 +388,5 @@
       <child link="right_link5_1"/>
       <axis xyz="0.0 0.0 -1.0"/>
-      <limit velocity="4.8" effort="30" lower="${-pi*2.0}" upper="${pi*2.0}" />
+      <limit velocity="4.8" effort="30" lower="${-pi*0.5}" upper="${pi*0.5}" />
       <dynamics damping="0.1" />
     </joint>
@@ -395,6 +395,6 @@
       <parent link="right_link5_1"/>
       <child link="right_link6_1"/>
-      <axis xyz="0.0 1.0 0.0"/>
-      <limit velocity="4.8" effort="30" lower="${-pi*2.0}" upper="${pi*2.0}" />
+      <axis xyz="0.0 -1.0 0.0"/>
+      <limit velocity="4.8" effort="30" lower="${-pi*0.5}" upper="${pi*0.5}" />
       <dynamics damping="0.1" />
     </joint>
@@ -403,6 +403,6 @@
       <parent link="right_link6_1"/>
       <child link="right_link_gripper_1"/>
-      <axis xyz="1.0 -0.0 -0.0"/>
-      <limit velocity="4.8" effort="30" lower="${-pi*2.0}" upper="${pi*2.0}" />
+      <axis xyz="1.0 0.0 0.0"/>
+      <limit velocity="4.8" effort="30" lower="${-pi*0.5}" upper="${pi*0.5}" />
       <dynamics damping="0.1" />
     </joint>
@@ -412,5 +412,5 @@
       <child link="left_link1_1"/>
       <axis xyz="0.0 1.0 0.0"/>
-      <limit velocity="4.8" effort="30" lower="${-pi*2.0}" upper="${pi*2.0}" />
+      <limit velocity="4.8" effort="30" lower="${-pi*0.5}" upper="${pi*0.5}" />
       <dynamics damping="0.1" />
     </joint>
@@ -419,6 +419,6 @@
       <parent link="left_link1_1"/>
       <child link="left_link2_1"/>
-      <axis xyz="-1.0 -0.0 -0.0"/>
-      <limit velocity="4.8" effort="30" lower="${-pi*2.0}" upper="${pi*2.0}" />
+      <axis xyz="1.0 0.0 0.0"/>
+      <limit velocity="4.8" effort="30" lower="${-pi*0.5}" upper="${pi*0.5}" />
       <dynamics damping="0.1" />
     </joint>
@@ -427,6 +427,6 @@
       <parent link="left_link2_1"/>
       <child link="left_link3_1"/>
-      <axis xyz="0.0 -0.0 -1.0"/>
-      <limit velocity="4.8" effort="30" lower="${-pi*2.0}" upper="${pi*2.0}" />
+      <axis xyz="0.0 0.0 -1.0"/>
+      <limit velocity="4.8" effort="30" lower="${-pi*0.5}" upper="${pi*0.5}" />
       <dynamics damping="0.1" />
     </joint>
@@ -435,6 +435,6 @@
       <parent link="left_link3_1"/>
       <child link="left_link4_1"/>
-      <axis xyz="-0.0 -1.0 0.0"/>
-      <limit velocity="4.8" effort="30" lower="${-pi*2.0}" upper="${pi*2.0}" />
+      <axis xyz="0.0 1.0 0.0"/>
+      <limit velocity="4.8" effort="30" lower="${-pi*0.5}" upper="${pi*0.5}" />
       <dynamics damping="0.1" />
     </joint>
@@ -444,5 +444,5 @@
       <child link="left_link5_1"/>
       <axis xyz="0.0 0.0 -1.0"/>
-      <limit velocity="4.8" effort="30" lower="${-pi*2.0}" upper="${pi*2.0}" />
+      <limit velocity="4.8" effort="30" lower="${-pi*0.5}" upper="${pi*0.5}" />
       <dynamics damping="0.1" />
     </joint>
@@ -451,6 +451,6 @@
       <parent link="left_link5_1"/>
       <child link="left_link6_1"/>
-      <axis xyz="-0.0 -1.0 -0.0"/>
-      <limit velocity="4.8" effort="30" lower="${-pi*2.0}" upper="${pi*2.0}" />
+      <axis xyz="0.0 1.0 0.0"/>
+      <limit velocity="4.8" effort="30" lower="${-pi*0.5}" upper="${pi*0.5}" />
       <dynamics damping="0.1" />
     </joint>
@@ -459,6 +459,6 @@
       <parent link="left_link6_1"/>
       <child link="left_link_gripper_1"/>
-      <axis xyz="1.0 -0.0 -0.0"/>
-      <limit velocity="4.8" effort="30" lower="${-pi*2.0}" upper="${pi*2.0}" />
+      <axis xyz="1.0 0.0 0.0"/>
+      <limit velocity="4.8" effort="30" lower="${-pi*0.5}" upper="${pi*0.5}" />
       <dynamics damping="0.1" />
     </joint>
@@ -467,6 +467,6 @@
       <parent link="base_link"/>
       <child link="neck_link1_1"/>
-      <axis xyz="0.0 1.0 -0.0"/>
-      <limit velocity="4.8" effort="30" lower="${-pi*2.0}" upper="${pi*2.0}" />
+      <axis xyz="0.0 -1.0 0.0"/>
+      <limit velocity="4.8" effort="30" lower="${-pi*0.5}" upper="${pi*0.5}" />
       <dynamics damping="0.1" />
     </joint>
@@ -476,5 +476,5 @@
       <child link="neck_link2_1"/>
       <axis xyz="0.0 0.0 1.0"/>
-      <limit velocity="4.8" effort="30" lower="${-pi*2.0}" upper="${pi*2.0}" />
+      <limit velocity="4.8" effort="30" lower="${-pi*0.5}" upper="${pi*0.5}" />
       <dynamics damping="0.1" />
     </joint>

Commit message: Edit joint axis

File: avatar_description/urdf/follower/follower_arm.urdf.xacro (robot description, xacro)
@@ -363,5 +363,5 @@
       <parent link="right_link1_1"/>
       <child link="right_link2_1"/>
-      <axis xyz="-1.0 0.0 0.0"/>
+      <axis xyz="1.0 0.0 0.0"/>
       <limit velocity="4.8" effort="30" lower="${-pi*0.5}" upper="${pi*0.5}" />
       <dynamics damping="0.1" />

Commit message: 충돌 감지 모든 부분 추가 (테스트 필요)

File: avatar_description/urdf/follower/follower_arm.urdf.xacro (robot description, xacro)
@@ -24,5 +24,5 @@
         <material name="dark_gray"/>
       </visual>
-      <collision>
+      <collision name="${prefix}base_link_collision">
         <origin xyz="0 0 0" rpy="0 0 0"/>
         <geometry>
@@ -45,5 +45,5 @@
         <material name="dark_gray"/>
       </visual>
-      <collision>
+      <collision name="${prefix}left_link1_1_collision">
         <origin xyz="0.00025 -0.1025 -0.6155" rpy="0 0 0"/>
         <geometry>
@@ -66,5 +66,5 @@
         <material name="dark_gray"/>
       </visual>
-      <collision>
+      <collision name="${prefix}right_link1_1_collision">
         <origin xyz="-0.00025 0.1025 -0.6155" rpy="0 0 0"/>
         <geometry>
@@ -87,5 +87,5 @@
         <material name="dark_gray"/>
       </visual>
-      <collision>
+      <collision name="${prefix}neck_link1_1_collision">
         <origin xyz="-0.00025 -0.0194 -0.6478" rpy="0 0 0"/>
         <geometry>
@@ -108,5 +108,5 @@
         <material name="white"/>
       </visual>
-      <collision>
+      <collision name="${prefix}neck_link2_1_collision">
         <origin xyz="-0.00025 -0.0004 -0.70755" rpy="0 0 0"/>
         <geometry>
@@ -129,5 +129,5 @@
         <material name="dark_gray"/>
       </visual>
-      <collision>
+      <collision name="${prefix}left_link2_1_collision">
         <origin xyz="-0.02425 -0.1525 -0.6155" rpy="0 0 0"/>
         <geometry>
@@ -150,5 +150,5 @@
         <material name="dark_gray"/>
       </visual>
-      <collision>
+      <collision name="${prefix}left_link3_1_collision">
         <origin xyz="0.00025 -0.1525 -0.45775" rpy="0 0 0"/>
         <geometry>
@@ -171,5 +171,5 @@
         <material name="dark_gray"/>
       </visual>
-      <collision>
+      <collision name="${prefix}left_link4_1_collision">
         <origin xyz="0.00025 -0.1715 -0.42625" rpy="0 0 0"/>
         <geometry>
@@ -192,5 +192,5 @@
         <material name="dark_gray"/>
       </visual>
-      <collision>
+      <collision name="${prefix}left_link5_1_collision">
         <origin xyz="0.00025 -0.1525 -0.28615" rpy="0 0 0"/>
         <geometry>
@@ -213,5 +213,5 @@
         <material name="dark_gray"/>
       </visual>
-      <collision>
+      <collision name="${prefix}left_link6_1_collision">
         <origin xyz="0.00025 -0.1715 -0.25465" rpy="0 0 0"/>
         <geometry>
@@ -255,5 +255,5 @@
         <material name="dark_gray"/>
       </visual>
-      <collision>
+      <collision name="${prefix}right_link2_1_collision">
         <origin xyz="-0.02475 0.1525 -0.6155" rpy="0 0 0"/>
         <geometry>
@@ -276,5 +276,5 @@
         <material name="dark_gray"/>
       </visual>
-      <collision>
+      <collision name="${prefix}right_link3_1_collision">
         <origin xyz="-0.00025 0.1525 -0.45775" rpy="0 0 0"/>
         <geometry>
@@ -297,5 +297,5 @@
         <material name="dark_gray"/>
       </visual>
-      <collision>
+      <collision name="${prefix}right_link4_1_collision">
         <origin xyz="-0.00025 0.1715 -0.42625" rpy="0 0 0"/>
         <geometry>
@@ -318,5 +318,5 @@
         <material name="dark_gray"/>
       </visual>
-      <collision>
+      <collision name="${prefix}right_link5_1_collision">
         <origin xyz="-0.00025 0.1525 -0.28615" rpy="0 0 0"/>
         <geometry>
@@ -339,5 +339,5 @@
         <material name="dark_gray"/>
       </visual>
-      <collision>
+      <collision name="${prefix}right_link6_1_collision">
         <origin xyz="-0.00025 0.1715 -0.25465" rpy="0 0 0"/>
         <geometry>
@@ -496,4 +496,125 @@
       <dynamics damping="0.1" />
     </joint>
+    <!-- Contact sensors for collision detection -->
+    <gazebo reference="base_link">
+      <sensor name="base_link_bumper" type="contact">
+        <always_on>true</always_on>
+        <update_rate>50.0</update_rate>
+        <contact>
+          <collision>${prefix}base_link_collision</collision>
+        </contact>
+        <plugin filename="libignition-gazebo-contact-system.so"
+                name="ignition::gazebo::systems::Contact">
+        </plugin>
+      </sensor>
+    </gazebo>
+    <gazebo reference="left_link1_1">
+      <sensor name="left_link1_1_bumper" type="contact">
+        <always_on>true</always_on>
+        <update_rate>50.0</update_rate>
+        <contact>
+          <collision>${prefix}left_link1_1_collision</collision>
+        </contact>
+        <plugin filename="libignition-gazebo-contact-system.so"
+                name="ignition::gazebo::systems::Contact">
+        </plugin>
+      </sensor>
+    </gazebo>
+    <gazebo reference="right_link1_1">
+      <sensor name="right_link1_1_bumper" type="contact">
+        <always_on>true</always_on>
+        <update_rate>50.0</update_rate>
+        <contact>
+          <collision>${prefix}right_link1_1_collision</collision>
+        </contact>
+        <plugin filename="libignition-gazebo-contact-system.so"
+                name="ignition::gazebo::systems::Contact">
+        </plugin>
+      </sensor>
+    </gazebo>
+    <gazebo reference="neck_link1_1">
+      <sensor name="neck_link1_1_bumper" type="contact">
+        <always_on>true</always_on>
+        <update_rate>50.0</update_rate>
+        <contact>
+          <collision>${prefix}neck_link1_1_collision</collision>
+        </contact>
+        <plugin filename="libignition-gazebo-contact-system.so"
+                name="ignition::gazebo::systems::Contact">
+        </plugin>
+      </sensor>
+    </gazebo>
+    <gazebo reference="neck_link2_1">
+      <sensor name="neck_link2_1_bumper" type="contact">
+        <always_on>true</always_on>
+        <update_rate>50.0</update_rate>
+        <contact>
+          <collision>${prefix}neck_link2_1_collision</collision>
+        </contact>
+        <plugin filename="libignition-gazebo-contact-system.so"
+                name="ignition::gazebo::systems::Contact">
+        </plugin>
+      </sensor>
+    </gazebo>
+    <gazebo reference="left_link2_1">
+      <sensor name="left_link2_1_bumper" type="contact">
+        <always_on>true</always_on>
+        <update_rate>50.0</update_rate>
+        <contact>
+          <collision>${prefix}left_link2_1_collision</collision>
+        </contact>
+        <plugin filename="libignition-gazebo-contact-system.so"
+                name="ignition::gazebo::systems::Contact">
+        </plugin>
+      </sensor>
+    </gazebo>
+    <gazebo reference="left_link3_1">
+      <sensor name="left_link3_1_bumper" type="contact">
+        <always_on>true</always_on>
+        <update_rate>50.0</update_rate>
+        <contact>
+          <collision>${prefix}left_link3_1_collision</collision>
+        </contact>
+        <plugin filename="libignition-gazebo-contact-system.so"
+                name="ignition::gazebo::systems::Contact">
+        </plugin>
+      </sensor>
+    </gazebo>
+    <gazebo reference="left_link4_1">
+      <sensor name="left_link4_1_bumper" type="contact">
+        <always_on>true</always_on>
+        <update_rate>50.0</update_rate>
+        <contact>
+          <collision>${prefix}left_link4_1_collision</collision>
+        </contact>
+        <plugin filename="libignition-gazebo-contact-system.so"
+                name="ignition::gazebo::systems::Contact">
+        </plugin>
+      </sensor>
+    </gazebo>
+    <gazebo reference="left_link5_1">
+      <sensor name="left_link5_1_bumper" type="contact">
+        <always_on>true</always_on>
+        <update_rate>50.0</update_rate>
+        <contact>
+          <collision>${prefix}left_link5_1_collision</collision>
+        </contact>
+        <plugin filename="libignition-gazebo-contact-system.so"
+                name="ignition::gazebo::systems::Contact">
+        </plugin>
+      </sensor>
+    </gazebo>
+    <gazebo reference="left_link6_1">
+      <sensor name="left_link6_1_bumper" type="contact">
+        <always_on>true</always_on>
+        <update_rate>50.0</update_rate>
+        <contact>
+          <collision>${prefix}left_link6_1_collision</collision>
+        </contact>
+        <plugin filename="libignition-gazebo-contact-system.so"
+                name="ignition::gazebo::systems::Contact">
+        </plugin>
+      </sensor>
+    </gazebo>
     <gazebo reference="left_link_gripper_1">
       <sensor name="left_gripper_bumper" type="contact">
@@ -501,5 +622,65 @@
         <update_rate>50.0</update_rate>
         <contact>
-          <collision>${prefix}left_link_gripper_1_collision_collision</collision>
+          <collision>${prefix}left_link_gripper_1_collision</collision>
+        </contact>
+        <plugin filename="libignition-gazebo-contact-system.so"
+                name="ignition::gazebo::systems::Contact">
+        </plugin>
+      </sensor>
+    </gazebo>
+    <gazebo reference="right_link2_1">
+      <sensor name="right_link2_1_bumper" type="contact">
+        <always_on>true</always_on>
+        <update_rate>50.0</update_rate>
+        <contact>
+          <collision>${prefix}right_link2_1_collision</collision>
+        </contact>
+        <plugin filename="libignition-gazebo-contact-system.so"
+                name="ignition::gazebo::systems::Contact">
+        </plugin>
+      </sensor>
+    </gazebo>
+    <gazebo reference="right_link3_1">
+      <sensor name="right_link3_1_bumper" type="contact">
+        <always_on>true</always_on>
+        <update_rate>50.0</update_rate>
+        <contact>
+          <collision>${prefix}right_link3_1_collision</collision>
+        </contact>
+        <plugin filename="libignition-gazebo-contact-system.so"
+                name="ignition::gazebo::systems::Contact">
+        </plugin>
+      </sensor>
+    </gazebo>
+    <gazebo reference="right_link4_1">
+      <sensor name="right_link4_1_bumper" type="contact">
+        <always_on>true</always_on>
+        <update_rate>50.0</update_rate>
+        <contact>
+          <collision>${prefix}right_link4_1_collision</collision>
+        </contact>
+        <plugin filename="libignition-gazebo-contact-system.so"
+                name="ignition::gazebo::systems::Contact">
+        </plugin>
+      </sensor>
+    </gazebo>
+    <gazebo reference="right_link5_1">
+      <sensor name="right_link5_1_bumper" type="contact">
+        <always_on>true</always_on>
+        <update_rate>50.0</update_rate>
+        <contact>
+          <collision>${prefix}right_link5_1_collision</collision>
+        </contact>
+        <plugin filename="libignition-gazebo-contact-system.so"
+                name="ignition::gazebo::systems::Contact">
+        </plugin>
+      </sensor>
+    </gazebo>
+    <gazebo reference="right_link6_1">
+      <sensor name="right_link6_1_bumper" type="contact">
+        <always_on>true</always_on>
+        <update_rate>50.0</update_rate>
+        <contact>
+          <collision>${prefix}right_link6_1_collision</collision>
         </contact>
         <plugin filename="libignition-gazebo-contact-system.so"
@@ -513,5 +694,5 @@
         <update_rate>50.0</update_rate>
         <contact>
-          <collision>${prefix}right_link_gripper_1_collision_collision</collision>
+          <collision>${prefix}right_link_gripper_1_collision</collision>
         </contact>
         <plugin filename="libignition-gazebo-contact-system.so"

Commit message: Edit neck axis

File: avatar_description/urdf/follower/follower_arm.urdf.xacro (robot description, xacro)
@@ -467,5 +467,5 @@
       <parent link="base_link"/>
       <child link="neck_link1_1"/>
-      <axis xyz="0.0 -1.0 0.0"/>
+      <axis xyz="0.0 1.0 0.0"/>
       <limit velocity="4.8" effort="30" lower="${-pi*0.5}" upper="${pi*0.5}" />
       <dynamics damping="0.1" />

Commit message: collision 변경

File: avatar_description/urdf/follower/follower_arm.urdf.xacro (robot description, xacro)
@@ -47,5 +47,5 @@
         <origin xyz="0.00025 -0.1025 -0.6155" rpy="0 0 0"/>
         <geometry>
-          <mesh filename="file://$(find avatar_description)/meshes/follower/left_link1_1.stl" scale="0.01 0.01 0.01"/>
+          <cylinder length="0.4" radius="0.05"/>
         </geometry>
       </collision>
@@ -67,5 +67,5 @@
         <origin xyz="-0.00025 0.1025 -0.6155" rpy="0 0 0"/>
         <geometry>
-          <mesh filename="file://$(find avatar_description)/meshes/follower/right_link1_1.stl" scale="0.01 0.01 0.01"/>
+          <cylinder length="0.4" radius="0.05"/>
         </geometry>
       </collision>
@@ -87,5 +87,5 @@
         <origin xyz="-0.00025 -0.0194 -0.6478" rpy="0 0 0"/>
         <geometry>
-          <mesh filename="file://$(find avatar_description)/meshes/follower/neck_link1_1.stl" scale="0.01 0.01 0.01"/>
+          <cylinder length="0.4" radius="0.05"/>
         </geometry>
       </collision>
@@ -107,5 +107,5 @@
         <origin xyz="-0.00025 -0.0004 -0.70755" rpy="0 0 0"/>
         <geometry>
-          <mesh filename="file://$(find avatar_description)/meshes/follower/neck_link2_1.stl" scale="0.01 0.01 0.01"/>
+          <cylinder length="0.4" radius="0.05"/>
         </geometry>
       </collision>
@@ -127,5 +127,5 @@
         <origin xyz="-0.02425 -0.1525 -0.6155" rpy="0 0 0"/>
         <geometry>
-          <mesh filename="file://$(find avatar_description)/meshes/follower/left_link2_1.stl" scale="0.01 0.01 0.01"/>
+          <cylinder length="0.4" radius="0.05"/>
         </geometry>
       </collision>
@@ -147,5 +147,5 @@
         <origin xyz="0.00025 -0.1525 -0.45775" rpy="0 0 0"/>
         <geometry>
-          <mesh filename="file://$(find avatar_description)/meshes/follower/left_link3_1.stl" scale="0.01 0.01 0.01"/>
+          <cylinder length="0.4" radius="0.05"/>
         </geometry>
       </collision>
@@ -167,5 +167,5 @@
         <origin xyz="0.00025 -0.1715 -0.42625" rpy="0 0 0"/>
         <geometry>
-          <mesh filename="file://$(find avatar_description)/meshes/follower/left_link4_1.stl" scale="0.01 0.01 0.01"/>
+          <cylinder length="0.4" radius="0.05"/>
         </geometry>
       </collision>
@@ -187,5 +187,5 @@
         <origin xyz="0.00025 -0.1525 -0.28615" rpy="0 0 0"/>
         <geometry>
-          <mesh filename="file://$(find avatar_description)/meshes/follower/left_link5_1.stl" scale="0.01 0.01 0.01"/>
+          <cylinder length="0.4" radius="0.05"/>
         </geometry>
       </collision>
@@ -207,5 +207,5 @@
         <origin xyz="0.00025 -0.1715 -0.25465" rpy="0 0 0"/>
         <geometry>
-          <mesh filename="file://$(find avatar_description)/meshes/follower/left_link6_1.stl" scale="0.01 0.01 0.01"/>
+          <cylinder length="0.4" radius="0.05"/>
         </geometry>
       </collision>
@@ -227,5 +227,5 @@
         <origin xyz="-0.01875 -0.1629 -0.20515" rpy="0 0 0"/>
         <geometry>
-          <mesh filename="file://$(find avatar_description)/meshes/follower/left_link_gripper_1.stl" scale="0.01 0.01 0.01"/>
+          <cylinder length="0.4" radius="0.05"/>
         </geometry>
       </collision>
@@ -247,5 +247,5 @@
         <origin xyz="-0.02475 0.1525 -0.6155" rpy="0 0 0"/>
         <geometry>
-          <mesh filename="file://$(find avatar_description)/meshes/follower/right_link2_1.stl" scale="0.01 0.01 0.01"/>
+          <cylinder length="0.4" radius="0.05"/>
         </geometry>
       </collision>
@@ -267,5 +267,5 @@
         <origin xyz="-0.00025 0.1525 -0.45775" rpy="0 0 0"/>
         <geometry>
-          <mesh filename="file://$(find avatar_description)/meshes/follower/right_link3_1.stl" scale="0.01 0.01 0.01"/>
+          <cylinder length="0.4" radius="0.05"/>
         </geometry>
       </collision>
@@ -287,5 +287,5 @@
         <origin xyz="-0.00025 0.1715 -0.42625" rpy="0 0 0"/>
         <geometry>
-          <mesh filename="file://$(find avatar_description)/meshes/follower/right_link4_1.stl" scale="0.01 0.01 0.01"/>
+          <cylinder length="0.4" radius="0.05"/>
         </geometry>
       </collision>
@@ -307,5 +307,5 @@
         <origin xyz="-0.00025 0.1525 -0.28615" rpy="0 0 0"/>
         <geometry>
-          <mesh filename="file://$(find avatar_description)/meshes/follower/right_link5_1.stl" scale="0.01 0.01 0.01"/>
+          <cylinder length="0.4" radius="0.05"/>
         </geometry>
       </collision>
@@ -327,5 +327,5 @@
         <origin xyz="-0.00025 0.1715 -0.25465" rpy="0 0 0"/>
         <geometry>
-          <mesh filename="file://$(find avatar_description)/meshes/follower/right_link6_1.stl" scale="0.01 0.01 0.01"/>
+          <cylinder length="0.4" radius="0.05"/>
         </geometry>
       </collision>
@@ -347,5 +347,5 @@
         <origin xyz="-0.01925 0.1645 -0.20515" rpy="0 0 0"/>
         <geometry>
-          <mesh filename="file://$(find avatar_description)/meshes/follower/right_link_gripper_1.stl" scale="0.01 0.01 0.01"/>
+          <cylinder length="0.4" radius="0.05"/>
         </geometry>
       </collision>
