Commit message: collision mesh형태도 표시됨을 확인

File: avatar_description/urdf/follower/follower_arm.urdf.xacro (robot description, xacro)
@@ -47,5 +47,5 @@
         <origin xyz="0.00025 -0.1025 -0.6155" rpy="0 0 0"/>
         <geometry>
-          <cylinder length="0.4" radius="0.05"/>
+          <mesh filename="file://$(find avatar_description)/meshes/follower/left_link1_1.stl" scale="0.01 0.01 0.01"/>
         </geometry>
       </collision>
@@ -67,5 +67,5 @@
         <origin xyz="-0.00025 0.1025 -0.6155" rpy="0 0 0"/>
         <geometry>
-          <cylinder length="0.4" radius="0.05"/>
+          <mesh filename="file://$(find avatar_description)/meshes/follower/right_link1_1.stl" scale="0.01 0.01 0.01"/>
         </geometry>
       </collision>
@@ -87,5 +87,5 @@
         <origin xyz="-0.00025 -0.0194 -0.6478" rpy="0 0 0"/>
         <geometry>
-          <cylinder length="0.4" radius="0.05"/>
+          <mesh filename="file://$(find avatar_description)/meshes/follower/neck_link1_1.stl" scale="0.01 0.01 0.01"/>
         </geometry>
       </collision>
@@ -107,5 +107,5 @@
         <origin xyz="-0.00025 -0.0004 -0.70755" rpy="0 0 0"/>
         <geometry>
-          <cylinder length="0.4" radius="0.05"/>
+          <mesh filename="file://$(find avatar_description)/meshes/follower/neck_link2_1.stl" scale="0.01 0.01 0.01"/>
         </geometry>
       </collision>
@@ -127,5 +127,5 @@
         <origin xyz="-0.02425 -0.1525 -0.6155" rpy="0 0 0"/>
         <geometry>
-          <cylinder length="0.4" radius="0.05"/>
+          <mesh filename="file://$(find avatar_description)/meshes/follower/left_link2_1.stl" scale="0.01 0.01 0.01"/>
         </geometry>
       </collision>
@@ -147,5 +147,5 @@
         <origin xyz="0.00025 -0.1525 -0.45775" rpy="0 0 0"/>
         <geometry>
-          <cylinder length="0.4" radius="0.05"/>
+          <mesh filename="file://$(find avatar_description)/meshes/follower/left_link3_1.stl" scale="0.01 0.01 0.01"/>
         </geometry>
       </collision>
@@ -167,5 +167,5 @@
         <origin xyz="0.00025 -0.1715 -0.42625" rpy="0 0 0"/>
         <geometry>
-          <cylinder length="0.4" radius="0.05"/>
+          <mesh filename="file://$(find avatar_description)/meshes/follower/left_link4_1.stl" scale="0.01 0.01 0.01"/>
         </geometry>
       </collision>
@@ -187,5 +187,5 @@
         <origin xyz="0.00025 -0.1525 -0.28615" rpy="0 0 0"/>
         <geometry>
-          <cylinder length="0.4" radius="0.05"/>
+          <mesh filename="file://$(find avatar_description)/meshes/follower/left_link5_1.stl" scale="0.01 0.01 0.01"/>
         </geometry>
       </collision>
@@ -207,5 +207,5 @@
         <origin xyz="0.00025 -0.1715 -0.25465" rpy="0 0 0"/>
         <geometry>
-          <cylinder length="0.4" radius="0.05"/>
+          <mesh filename="file://$(find avatar_description)/meshes/follower/left_link6_1.stl" scale="0.01 0.01 0.01"/>
         </geometry>
       </collision>
@@ -227,5 +227,5 @@
         <origin xyz="-0.01875 -0.1629 -0.20515" rpy="0 0 0"/>
         <geometry>
-          <cylinder length="0.4" radius="0.05"/>
+          <mesh filename="file://$(find avatar_description)/meshes/follower/left_link_gripper_1.stl" scale="0.01 0.01 0.01"/>
         </geometry>
       </collision>
@@ -247,5 +247,5 @@
         <origin xyz="-0.02475 0.1525 -0.6155" rpy="0 0 0"/>
         <geometry>
-          <cylinder length="0.4" radius="0.05"/>
+          <mesh filename="file://$(find avatar_description)/meshes/follower/right_link2_1.stl" scale="0.01 0.01 0.01"/>
         </geometry>
       </collision>
@@ -267,5 +267,5 @@
         <origin xyz="-0.00025 0.1525 -0.45775" rpy="0 0 0"/>
         <geometry>
-          <cylinder length="0.4" radius="0.05"/>
+          <mesh filename="file://$(find avatar_description)/meshes/follower/right_link3_1.stl" scale="0.01 0.01 0.01"/>
         </geometry>
       </collision>
@@ -287,5 +287,5 @@
         <origin xyz="-0.00025 0.1715 -0.42625" rpy="0 0 0"/>
         <geometry>
-          <cylinder length="0.4" radius="0.05"/>
+          <mesh filename="file://$(find avatar_description)/meshes/follower/right_link4_1.stl" scale="0.01 0.01 0.01"/>
         </geometry>
       </collision>
@@ -307,5 +307,5 @@
         <origin xyz="-0.00025 0.1525 -0.28615" rpy="0 0 0"/>
         <geometry>
-          <cylinder length="0.4" radius="0.05"/>
+          <mesh filename="file://$(find avatar_description)/meshes/follower/right_link5_1.stl" scale="0.01 0.01 0.01"/>
         </geometry>
       </collision>
@@ -327,5 +327,5 @@
         <origin xyz="-0.00025 0.1715 -0.25465" rpy="0 0 0"/>
         <geometry>
-          <cylinder length="0.4" radius="0.05"/>
+          <mesh filename="file://$(find avatar_description)/meshes/follower/right_link6_1.stl" scale="0.01 0.01 0.01"/>
         </geometry>
       </collision>
@@ -347,5 +347,5 @@
         <origin xyz="-0.01925 0.1645 -0.20515" rpy="0 0 0"/>
         <geometry>
-          <cylinder length="0.4" radius="0.05"/>
+          <mesh filename="file://$(find avatar_description)/meshes/follower/right_link_gripper_1.stl" scale="0.01 0.01 0.01"/>
         </geometry>
       </collision>

Commit message: 4,6 joint 가제보 제한

File: avatar_description/urdf/follower/follower_arm.urdf.xacro (robot description, xacro)
@@ -380,5 +380,5 @@
       <child link="${prefix}right_link4_1"/>
       <axis xyz="0.0 -1.0 -0.0"/>
-      <limit velocity="4.8" effort="30" lower="${-pi*2.0}" upper="${pi*2.0}" />
+      <limit velocity="4.8" effort="30" lower="${-pi*0.389}" upper="${pi*0.389}" />
       <dynamics damping="0.1" />
     </joint>
@@ -396,5 +396,5 @@
       <child link="${prefix}right_link6_1"/>
       <axis xyz="0.0 -1.0 0.0"/>
-      <limit velocity="4.8" effort="30" lower="${-pi*2.0}" upper="${pi*2.0}" />
+      <limit velocity="4.8" effort="30" lower="${-pi*0.389}" upper="${pi*0.389}" />
       <dynamics damping="0.1" />
     </joint>
@@ -436,5 +436,5 @@
       <child link="${prefix}left_link4_1"/>
       <axis xyz="-0.0 1.0 0.0"/>
-      <limit velocity="4.8" effort="30" lower="${-pi*2.0}" upper="${pi*2.0}" />
+      <limit velocity="4.8" effort="30" lower="${-pi*0.389}" upper="${pi*0.389}" />
       <dynamics damping="0.1" />
     </joint>
@@ -452,5 +452,5 @@
       <child link="${prefix}left_link6_1"/>
       <axis xyz="-0.0 1.0 -0.0"/>
-      <limit velocity="4.8" effort="30" lower="${-pi*2.0}" upper="${pi*2.0}" />
+      <limit velocity="4.8" effort="30" lower="${-pi*0.389}" upper="${pi*0.389}" />
       <dynamics damping="0.1" />
     </joint>
