Commit message: Add new urdf

File: avatar_description/gazebo/follower.gazebo.xacro (robot description, xacro)
@@ -31,4 +31,5 @@
     <xacro:Link reference="${prefix}right_link5"/>
     <xacro:Link reference="${prefix}right_link6"/>
+    <xacro:Link reference="${prefix}right_link_gripper"/>
     <xacro:Link reference="${prefix}left_link1"/>
     <xacro:Link reference="${prefix}left_link2"/>
@@ -37,12 +38,23 @@
     <xacro:Link reference="${prefix}left_link5"/>
     <xacro:Link reference="${prefix}left_link6"/>
+    <xacro:Link reference="${prefix}left_link_gripper"/>
     <xacro:Link reference="${prefix}neck_link1"/>
     <xacro:Link reference="${prefix}neck_link2"/>
     <xacro:SimpleTransmission trans="${prefix}trans1" joint="${prefix}right_joint1" actuator="${prefix}actuator1" />
     <xacro:SimpleTransmission trans="${prefix}trans2" joint="${prefix}right_joint2" actuator="${prefix}actuator2" />
-    <xacro:SimpleTransmission trans="${prefix}trans3" joint="${prefix}right_joint2" actuator="${prefix}actuator3" />
-    <xacro:SimpleTransmission trans="${prefix}trans4" joint="${prefix}right_joint2" actuator="${prefix}actuator4" />
-    <xacro:SimpleTransmission trans="${prefix}trans5" joint="${prefix}right_joint2" actuator="${prefix}actuator5" />
-    <xacro:SimpleTransmission trans="${prefix}trans6" joint="${prefix}right_joint2" actuator="${prefix}actuator6" />
+    <xacro:SimpleTransmission trans="${prefix}trans3" joint="${prefix}right_joint3" actuator="${prefix}actuator3" />
+    <xacro:SimpleTransmission trans="${prefix}trans4" joint="${prefix}right_joint4" actuator="${prefix}actuator4" />
+    <xacro:SimpleTransmission trans="${prefix}trans5" joint="${prefix}right_joint5" actuator="${prefix}actuator5" />
+    <xacro:SimpleTransmission trans="${prefix}trans6" joint="${prefix}right_joint6" actuator="${prefix}actuator6" />
+    <xacro:SimpleTransmission trans="${prefix}trans7" joint="${prefix}right_gripper_joint" actuator="${prefix}actuator7" />
+    <xacro:SimpleTransmission trans="${prefix}trans8" joint="${prefix}left_joint1" actuator="${prefix}actuator8" />
+    <xacro:SimpleTransmission trans="${prefix}trans9" joint="${prefix}left_joint2" actuator="${prefix}actuator9" />
+    <xacro:SimpleTransmission trans="${prefix}trans10" joint="${prefix}left_joint3" actuator="${prefix}actuator10" />
+    <xacro:SimpleTransmission trans="${prefix}trans11" joint="${prefix}left_joint4" actuator="${prefix}actuator11" />
+    <xacro:SimpleTransmission trans="${prefix}trans12" joint="${prefix}left_joint5" actuator="${prefix}actuator12" />
+    <xacro:SimpleTransmission trans="${prefix}trans13" joint="${prefix}left_joint6" actuator="${prefix}actuator13" />
+    <xacro:SimpleTransmission trans="${prefix}trans14" joint="${prefix}left_gripper_joint" actuator="${prefix}actuator14" />
+    <xacro:SimpleTransmission trans="${prefix}trans15" joint="${prefix}neck_joint1" actuator="${prefix}actuator15" />
+    <xacro:SimpleTransmission trans="${prefix}trans16" joint="${prefix}neck_joint2" actuator="${prefix}actuator16" />
   </xacro:macro>
 </robot>

File: avatar_description/ros2_control/follower.ros2_control.xacro (robot description, xacro)
@@ -102,4 +102,10 @@
         <param name="ID">16</param>
       </joint>
+      <joint name="${prefix}right_joint_gripper">
+        <command_interface name="position"/>
+        <state_interface name="position"/>
+        <state_interface name="velocity"/>
+        <param name="ID">17</param>
+      </joint>
       <!-- 왼쪽 팔 -->
       <joint name="${prefix}left_joint1">
@@ -138,4 +144,10 @@
         <state_interface name="velocity"/>
         <param name="ID">26</param>
+      </joint>
+      <joint name="${prefix}left_joint_gripper">
+        <command_interface name="position"/>
+        <state_interface name="position"/>
+        <state_interface name="velocity"/>
+        <param name="ID">27</param>
       </joint>
       <!-- neck joint -->
@@ -266,4 +278,23 @@
           <param name="Profile Acceleration">25</param>
         </gpio>
+        <gpio name="dxl16">
+          <param name="type">dxl</param>
+          <param name="ID">17</param>
+          <command_interface name="Goal Position"/>
+          <state_interface name="Present Position"/>
+          <state_interface name="Present Velocity"/>
+          <param name="Drive Mode">4</param>
+          <param name="Operating Mode">4</param>
+          <param name="Return Delay Time">0</param>
+          <param name="Min Position Limit">1024</param>
+          <param name="Max Position Limit">3140</param>
+          <param name="Min Position Limit">830</param>
+          <param name="Max Position Limit">3129</param>
+          <param name="Position P Gain">1000</param>
+          <param name="Position I Gain">0</param>
+          <param name="Position D Gain">1000</param>
+          <param name="Profile Velocity">50</param>
+          <param name="Profile Acceleration">25</param>
+        </gpio>
         <gpio name="dxl21">
           <param name="type">dxl</param>
@@ -364,4 +395,23 @@
           <param name="type">dxl</param>
           <param name="ID">26</param>
+          <command_interface name="Goal Position"/>
+          <state_interface name="Present Position"/>
+          <state_interface name="Present Velocity"/>
+          <param name="Drive Mode">4</param>
+          <param name="Operating Mode">4</param>
+          <param name="Return Delay Time">0</param>
+          <param name="Min Position Limit">1024</param>
+          <param name="Max Position Limit">3140</param>
+          <param name="Min Position Limit">830</param>
+          <param name="Max Position Limit">3129</param>
+          <param name="Position P Gain">1000</param>
+          <param name="Position I Gain">0</param>
+          <param name="Position D Gain">1000</param>
+          <param name="Profile Velocity">50</param>
+          <param name="Profile Acceleration">25</param>
+        </gpio>
+        <gpio name="dxl26">
+          <param name="type">dxl</param>
+          <param name="ID">27</param>
           <command_interface name="Goal Position"/>
           <state_interface name="Present Position"/>

File: avatar_description/urdf/follower/follower.urdf.xacro (robot description, xacro)
@@ -14,5 +14,5 @@
   <joint name="$(arg prefix)world_fixed" type="fixed">
     <parent link="world"/>
-    <child link="$(arg prefix)link0"/>
+    <child link="$(arg prefix)base_link"/>
     <origin xyz="0.0 0.0 0.0" rpy="0 0 0"/>
   </joint>

File: avatar_description/urdf/follower/follower_arm.urdf.xacro (robot description, xacro)
@@ -2,486 +2,449 @@
 <robot xmlns:xacro="http://www.ros.org/wiki/xacro">
   <xacro:macro name="follower" params="prefix">
-    <!-- <xacro:property name="pi" value="3.1415926535" /> -->
-    <xacro:property name="robot_thickness" value="0.08" />
-    <xacro:property name="body_height" value="0.5" />
-    <xacro:property name="body_width" value="0.4" />
-    <xacro:property name="arm1_height" value="0.15"/>
-    <xacro:property name="arm2_height" value="0.10"/>
-    <xacro:property name="gripper_height" value="0.05"/>
-    <!-- link0 -->
-    <link name="${prefix}link0" >
-      <visual>
-        <origin xyz="0 0 ${body_height/2}" rpy="0 0 0" />
-        <geometry>
-          <box size="${body_width} ${robot_thickness} ${body_height}" />
-          <!-- <mesh filename="${meshes_file_direction}/follower_01_base.stl" scale="0.001 0.001 0.001" /> -->
-        </geometry>
-        <material name="grey">
-          <color rgba="0.2 0.2 0.2 1" />
-        </material>
-      </visual>
-      <collision>
-        <origin xyz="0 0 ${body_height/2}" rpy="0 0 0" />
-        <geometry>
-          <box size="${body_width} ${robot_thickness} ${body_height}" />
-        </geometry>
-      </collision>
-      <inertial>
-        <origin xyz="0 0 0" />
-        <mass value="2.0e-1" />
-        <inertia ixx="1e-4" ixy="0" ixz="0" iyy="1e-4" iyz="0" izz="1e-4" />
-      </inertial>
-    </link>
-    <!-- right arm -->
-    <!-- joint1 -->
-    <joint name="${prefix}right_joint1" type="revolute">
-      <parent link="${prefix}link0" />
-      <child link="${prefix}right_link1" />
-      <origin xyz="${body_width/2} 0 ${body_height - robot_thickness/2}" rpy="0 0 0" />
-      <axis xyz="1 0 0" />
-      <limit velocity="4.8" effort="1000" lower="${-pi}" upper="${pi}" />
-      <dynamics damping="0.05" />
-    </joint>
-    <!-- link1 -->
-    <link name="${prefix}right_link1" >
-      <visual>
-        <origin xyz="${robot_thickness/2} 0 0" rpy="${pi/2} 0 0" />
-        <geometry>
-          <cylinder radius="${robot_thickness/2}" length="${robot_thickness}"/>
-        </geometry>
-        <material name="grey">
-          <color rgba="0.2 0.2 0.2 1" />
-        </material>
-      </visual>
-      <collision>
-        <origin xyz="${robot_thickness/2} 0 0" rpy="${pi/2} 0 0" />
-        <geometry>
-          <cylinder radius="${robot_thickness/2}" length="${robot_thickness}"/>
-        </geometry>
-      </collision>
-      <inertial>
-        <origin xyz="0 0 0.05" />
-        <mass value="1.0e-1" />
-        <inertia ixx="5e-5" ixy="0" ixz="0" iyy="5e-5" iyz="0" izz="1e-5" />
-      </inertial>
-    </link>
-    <!-- joint2 -->
-    <joint name="${prefix}right_joint2" type="revolute">
-      <parent link="${prefix}right_link1" />
-      <child link="${prefix}right_link2" />
-      <origin xyz="${robot_thickness/2} 0 0" rpy="0 0 0" />
-      <axis xyz="0 1 0" />
-      <limit velocity="4.8" effort="1000" lower="${-pi}" upper="${pi/2}" />
-      <dynamics damping="0.1" />
-    </joint>
-    <!-- link2 -->
-    <link name="${prefix}right_link2" >
-      <visual>
-        <origin xyz="0 0 ${-robot_thickness/2 - arm1_height/2}" rpy="0 0 0" />
-        <geometry>
-          <box size="${robot_thickness} ${robot_thickness} ${arm1_height}" />
-        </geometry>
-        <material name="grey">
-          <color rgba="0.2 0.2 0.2 1" />
-        </material>
-      </visual>
-      <collision>
-        <origin xyz="0 0 ${-robot_thickness/2 - arm1_height/2}" rpy="0 0 0" />
-        <geometry>
-          <box size="${robot_thickness} ${robot_thickness} ${arm1_height}" />
-        </geometry>
-      </collision>
-      <inertial>
-        <origin xyz="0 0 0.05" />
-        <mass value="8.0e-2" />
-        <inertia ixx="4e-5" ixy="0" ixz="0" iyy="4e-5" iyz="0" izz="8e-6" />
-      </inertial>
-    </link>
-    <!-- joint3 -->
-    <joint name="${prefix}right_joint3" type="revolute">
-      <parent link="${prefix}right_link2" />
-      <child link="${prefix}right_link3" />
-      <origin xyz="0 0 ${-arm1_height - robot_thickness/2}" rpy="0 0 0" />
-      <axis xyz="0 0 -1" />
-      <limit velocity="4.8" effort="1000" lower="${-pi/2}" upper="${pi/2}" />
-      <dynamics damping="0.1" />
-    </joint>
-    <!-- link3 -->
-    <link name="${prefix}right_link3" >
-      <visual>
-        <origin xyz="0 0 ${-robot_thickness/2}" rpy="${pi/2} 0 ${pi/2}" />
-        <geometry>
-          <cylinder radius="${robot_thickness/2}" length="${robot_thickness}"/>
-        </geometry>
-        <material name="grey">
-          <color rgba="0.2 0.2 0.2 1" />
-        </material>
-      </visual>
-      <collision>
-        <origin xyz="0 0 ${-robot_thickness/2}" rpy="${pi/2} 0 ${pi/2}" />
-        <geometry>
-          <cylinder radius="${robot_thickness/2}" length="${robot_thickness}"/>
-        </geometry>
-      </collision>
-      <inertial>
-        <origin xyz="0 0 0.05" />
-        <mass value="1.0e-1" />
-        <inertia ixx="5e-5" ixy="0" ixz="0" iyy="5e-5" iyz="0" izz="1e-5" />
-      </inertial>
-    </link>
-    <!-- joint4 -->
-    <joint name="${prefix}right_joint4" type="revolute">
-      <parent link="${prefix}right_link3" />
-      <child link="${prefix}right_link4" />
-      <origin xyz="0 0 ${-robot_thickness/2}" rpy="0 0 0" />
-      <axis xyz="1 0 0" />
-      <limit velocity="4.8" effort="1000" lower="0" upper="${pi}" />
-      <dynamics damping="0.1" />
-    </joint>
-    <!-- link4 -->
-    <link name="${prefix}right_link4" >
-      <visual>
-        <origin xyz="0 0 ${-robot_thickness/2 - arm2_height/2}" rpy="0 0 0" />
-        <geometry>
-          <box size="${robot_thickness} ${robot_thickness} ${arm2_height}" />
-        </geometry>
-        <material name="grey">
-          <color rgba="0.2 0.2 0.2 1" />
-        </material>
-      </visual>
-      <collision>
-        <origin xyz="0 0 ${-robot_thickness/2 - arm2_height/2}" rpy="0 0 0" />
-        <geometry>
-          <box size="${robot_thickness} ${robot_thickness} ${arm2_height}" />
-        </geometry>
-      </collision>
-      <inertial>
-        <origin xyz="0 0 0.05" />
-        <mass value="8.0e-2" />
-        <inertia ixx="4e-5" ixy="0" ixz="0" iyy="4e-5" iyz="0" izz="8e-6" />
-      </inertial>
-    </link>
-     <!-- joint5 -->
-    <joint name="${prefix}right_joint5" type="revolute">
-      <parent link="${prefix}right_link4" />
-      <child link="${prefix}right_link5" />
-      <origin xyz="0 0 ${-arm2_height - robot_thickness/2}" rpy="0 0 0" />
-      <axis xyz="0 0 -1" />
-      <limit velocity="4.8" effort="1000" lower="${-pi/2}" upper="${pi/2}" />
-      <dynamics damping="0.1" />
-    </joint>
-    <!-- link5 -->
-    <link name="${prefix}right_link5" >
-      <visual>
-        <origin xyz="0 0 ${-robot_thickness/2}" rpy="${pi/2} 0 ${pi/2}" />
-        <geometry>
-          <cylinder radius="${robot_thickness/2}" length="${robot_thickness}"/>
-        </geometry>
-        <material name="grey">
-          <color rgba="0.2 0.2 0.2 1" />
-        </material>
-      </visual>
-      <collision>
-        <origin xyz="0 0 ${-robot_thickness/2}" rpy="${pi/2} 0 ${pi/2}" />
-        <geometry>
-          <cylinder radius="${robot_thickness/2}" length="${robot_thickness}"/>
-        </geometry>
-      </collision>
-      <inertial>
-        <origin xyz="0 0 0.05" />
-        <mass value="1.0e-1" />
-        <inertia ixx="5e-5" ixy="0" ixz="0" iyy="5e-5" iyz="0" izz="1e-5" />
-      </inertial>
-    </link>
-    <!-- joint6 -->
-    <joint name="${prefix}right_joint6" type="revolute">
-      <parent link="${prefix}right_link5" />
-      <child link="${prefix}right_link6" />
-      <origin xyz="0 0 ${-robot_thickness/2}" rpy="0 0 0" />
-      <axis xyz="1 0 0" />
-      <limit velocity="4.8" effort="1000" lower="${-pi/2}" upper="${pi/2}" />
-      <dynamics damping="0.1" />
-    </joint>
-    <!-- link6 -->
-    <link name="${prefix}right_link6" >
-      <visual>
-        <origin xyz="0 0 ${-robot_thickness/2 - gripper_height/2}" rpy="0 0 0" />
-        <geometry>
-          <box size="${robot_thickness} ${robot_thickness} ${gripper_height}" />
-        </geometry>
-        <material name="grey">
-          <color rgba="0.2 0.2 0.2 1" />
-        </material>
-      </visual>
-      <collision>
-        <origin xyz="0 0 ${-robot_thickness/2 - gripper_height/2}" rpy="0 0 0" />
-        <geometry>
-          <box size="${robot_thickness} ${robot_thickness} ${gripper_height}" />
-        </geometry>
-      </collision>
-      <inertial>
-        <origin xyz="0 0 0.05" />
-        <mass value="8.0e-2" />
-        <inertia ixx="4e-5" ixy="0" ixz="0" iyy="4e-5" iyz="0" izz="8e-6" />
-      </inertial>
-    </link>
-    <!-- left arm -->
-    <!-- joint1 -->
-    <joint name="${prefix}left_joint1" type="revolute">
-      <parent link="${prefix}link0" />
-      <child link="${prefix}left_link1" />
-      <origin xyz="${-body_width/2} 0 ${body_height - robot_thickness/2}" rpy="0 0 0" />
-      <axis xyz="1 0 0" />
-      <limit velocity="4.8" effort="1000" lower="${-pi}" upper="${pi}" />
-      <dynamics damping="0.05" />
-    </joint>
-    <!-- link1 -->
-    <link name="${prefix}left_link1" >
-      <visual>
-        <origin xyz="${-robot_thickness/2} 0 0" rpy="${pi/2} 0 0" />
-        <geometry>
-          <cylinder radius="${robot_thickness/2}" length="${robot_thickness}"/>
-        </geometry>
-        <material name="grey">
-          <color rgba="0.2 0.2 0.2 1" />
-        </material>
-      </visual>
-      <collision>
-        <origin xyz="${-robot_thickness/2} 0 0" rpy="${pi/2} 0 0" />
-        <geometry>
-          <cylinder radius="${robot_thickness/2}" length="${robot_thickness}"/>
-        </geometry>
-      </collision>
-      <inertial>
-        <origin xyz="0 0 0.05" />
-        <mass value="1.0e-1" />
-        <inertia ixx="5e-5" ixy="0" ixz="0" iyy="5e-5" iyz="0" izz="1e-5" />
-      </inertial>
-    </link>
-    <!-- joint2 -->
-    <joint name="${prefix}left_joint2" type="revolute">
-      <parent link="${prefix}left_link1" />
-      <child link="${prefix}left_link2" />
-      <origin xyz="${-robot_thickness/2} 0 0" rpy="0 0 0" />
-      <axis xyz="0 1 0" />
-      <limit velocity="4.8" effort="1000" lower="${-pi/2}" upper="${pi}" />
-      <dynamics damping="0.1" />
-    </joint>
-    <!-- link2 -->
-    <link name="${prefix}left_link2" >
-      <visual>
-        <origin xyz="0 0 ${-robot_thickness/2 - arm1_height/2}" rpy="0 0 0" />
-        <geometry>
-          <box size="${robot_thickness} ${robot_thickness} ${arm1_height}" />
-        </geometry>
-        <material name="grey">
-          <color rgba="0.2 0.2 0.2 1" />
-        </material>
-      </visual>
-      <collision>
-        <origin xyz="0 0 ${-robot_thickness/2 - arm1_height/2}" rpy="0 0 0" />
-        <geometry>
-          <box size="${robot_thickness} ${robot_thickness} ${arm1_height}" />
-        </geometry>
-      </collision>
-      <inertial>
-        <origin xyz="0 0 0.05" />
-        <mass value="8.0e-2" />
-        <inertia ixx="4e-5" ixy="0" ixz="0" iyy="4e-5" iyz="0" izz="8e-6" />
-      </inertial>
-    </link>
-    <!-- joint3 -->
-    <joint name="${prefix}left_joint3" type="revolute">
-      <parent link="${prefix}left_link2" />
-      <child link="${prefix}left_link3" />
-      <origin xyz="0 0 ${-arm1_height - robot_thickness/2}" rpy="0 0 0" />
-      <axis xyz="0 0 -1" />
-      <limit velocity="4.8" effort="1000" lower="${-pi/2}" upper="${pi/2}" />
-      <dynamics damping="0.1" />
-    </joint>
-    <!-- link3 -->
-    <link name="${prefix}left_link3" >
-      <visual>
-        <origin xyz="0 0 ${-robot_thickness/2}" rpy="${pi/2} 0 ${pi/2}" />
-        <geometry>
-          <cylinder radius="${robot_thickness/2}" length="${robot_thickness}"/>
-        </geometry>
-        <material name="grey">
-          <color rgba="0.2 0.2 0.2 1" />
-        </material>
-      </visual>
-      <collision>
-        <origin xyz="0 0 ${-robot_thickness/2}" rpy="${pi/2} 0 ${pi/2}" />
-        <geometry>
-          <cylinder radius="${robot_thickness/2}" length="${robot_thickness}"/>
-        </geometry>
-      </collision>
-      <inertial>
-        <origin xyz="0 0 0.05" />
-        <mass value="1.0e-1" />
-        <inertia ixx="5e-5" ixy="0" ixz="0" iyy="5e-5" iyz="0" izz="1e-5" />
-      </inertial>
-    </link>
-    <!-- joint4 -->
-    <joint name="${prefix}left_joint4" type="revolute">
-      <parent link="${prefix}left_link3" />
-      <child link="${prefix}left_link4" />
-      <origin xyz="0 0 ${-robot_thickness/2}" rpy="0 0 0" />
-      <axis xyz="1 0 0" />
-      <limit velocity="4.8" effort="1000" lower="0" upper="${pi}" />
-      <dynamics damping="0.1" />
-    </joint>
-    <!-- link4 -->
-    <link name="${prefix}left_link4" >
-      <visual>
-        <origin xyz="0 0 ${-robot_thickness/2 - arm2_height/2}" rpy="0 0 0" />
-        <geometry>
-          <box size="${robot_thickness} ${robot_thickness} ${arm2_height}" />
-        </geometry>
-        <material name="grey">
-          <color rgba="0.2 0.2 0.2 1" />
-        </material>
-      </visual>
-      <collision>
-        <origin xyz="0 0 ${-robot_thickness/2 - arm2_height/2}" rpy="0 0 0" />
-        <geometry>
-          <box size="${robot_thickness} ${robot_thickness} ${arm2_height}" />
-        </geometry>
-      </collision>
-      <inertial>
-        <origin xyz="0 0 0.05" />
-        <mass value="8.0e-2" />
-        <inertia ixx="4e-5" ixy="0" ixz="0" iyy="4e-5" iyz="0" izz="8e-6" />
-      </inertial>
-    </link>
-     <!-- joint5 -->
-    <joint name="${prefix}left_joint5" type="revolute">
-      <parent link="${prefix}left_link4" />
-      <child link="${prefix}left_link5" />
-      <origin xyz="0 0 ${-arm2_height - robot_thickness/2}" rpy="0 0 0" />
-      <axis xyz="0 0 -1" />
-      <limit velocity="4.8" effort="1000" lower="${-pi/2}" upper="${pi/2}" />
-      <dynamics damping="0.1" />
-    </joint>
-    <!-- link5 -->
-    <link name="${prefix}left_link5" >
-      <visual>
-        <origin xyz="0 0 ${-robot_thickness/2}" rpy="${pi/2} 0 ${pi/2}" />
-        <geometry>
-          <cylinder radius="${robot_thickness/2}" length="${robot_thickness}"/>
-        </geometry>
-        <material name="grey">
-          <color rgba="0.2 0.2 0.2 1" />
-        </material>
-      </visual>
-      <collision>
-        <origin xyz="0 0 ${-robot_thickness/2}" rpy="${pi/2} 0 ${pi/2}" />
-        <geometry>
-          <cylinder radius="${robot_thickness/2}" length="${robot_thickness}"/>
-        </geometry>
-      </collision>
-      <inertial>
-        <origin xyz="0 0 0.05" />
-        <mass value="1.0e-1" />
-        <inertia ixx="5e-5" ixy="0" ixz="0" iyy="5e-5" iyz="0" izz="1e-5" />
-      </inertial>
-    </link>
-    <!-- joint6 -->
-    <joint name="${prefix}left_joint6" type="revolute">
-      <parent link="${prefix}left_link5" />
-      <child link="${prefix}left_link6" />
-      <origin xyz="0 0 ${-robot_thickness/2}" rpy="0 0 0" />
-      <axis xyz="1 0 0" />
-      <limit velocity="4.8" effort="1000" lower="${-pi/2}" upper="${pi/2}" />
-      <dynamics damping="0.1" />
-    </joint>
-    <!-- link6 -->
-    <link name="${prefix}left_link6" >
-      <visual>
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