Commit message: 충돌감지 수정 최종(이제 mesh 형태를 평범한 모습으로 바꾸면 굄)

File: avatar_description/gazebo/follower.gazebo.xacro (robot description, xacro)
@@ -24,21 +24,21 @@
       </gazebo>
     </xacro:macro>
-    <xacro:Link reference="${prefix}link0"/>
-    <xacro:Link reference="${prefix}right_link1"/>
-    <xacro:Link reference="${prefix}right_link2"/>
-    <xacro:Link reference="${prefix}right_link3"/>
-    <xacro:Link reference="${prefix}right_link4"/>
-    <xacro:Link reference="${prefix}right_link5"/>
-    <xacro:Link reference="${prefix}right_link6"/>
-    <xacro:Link reference="${prefix}right_link_gripper"/>
-    <xacro:Link reference="${prefix}left_link1"/>
-    <xacro:Link reference="${prefix}left_link2"/>
-    <xacro:Link reference="${prefix}left_link3"/>
-    <xacro:Link reference="${prefix}left_link4"/>
-    <xacro:Link reference="${prefix}left_link5"/>
-    <xacro:Link reference="${prefix}left_link6"/>
-    <xacro:Link reference="${prefix}left_link_gripper"/>
-    <xacro:Link reference="${prefix}neck_link1"/>
-    <xacro:Link reference="${prefix}neck_link2"/>
+    <xacro:Link reference="base_link"/>
+    <xacro:Link reference="${prefix}right_link1_1"/>
+    <xacro:Link reference="${prefix}right_link2_1"/>
+    <xacro:Link reference="${prefix}right_link3_1"/>
+    <xacro:Link reference="${prefix}right_link4_1"/>
+    <xacro:Link reference="${prefix}right_link5_1"/>
+    <xacro:Link reference="${prefix}right_link6_1"/>
+    <xacro:Link reference="${prefix}right_link_gripper_1"/>
+    <xacro:Link reference="${prefix}left_link1_1"/>
+    <xacro:Link reference="${prefix}left_link2_1"/>
+    <xacro:Link reference="${prefix}left_link3_1"/>
+    <xacro:Link reference="${prefix}left_link4_1"/>
+    <xacro:Link reference="${prefix}left_link5_1"/>
+    <xacro:Link reference="${prefix}left_link6_1"/>
+    <xacro:Link reference="${prefix}left_link_gripper_1"/>
+    <xacro:Link reference="${prefix}neck_link1_1"/>
+    <xacro:Link reference="${prefix}neck_link2_1"/>
     <xacro:SimpleTransmission trans="${prefix}trans1" joint="${prefix}right_joint1" actuator="${prefix}actuator1" />
     <xacro:SimpleTransmission trans="${prefix}trans2" joint="${prefix}right_joint2" actuator="${prefix}actuator2" />

File: avatar_description/urdf/follower/follower_arm.urdf.xacro (robot description, xacro)
@@ -11,5 +11,5 @@
       <color rgba="1.0 1.0 1.0 1.0"/>
     </material>
-    <link name="base_link">
+    <link name="${prefix}base_link">
       <inertial>
         <origin xyz="1.197034860872733e-05 2.2046610134709234e-05 0.13090240145620716" rpy="0 0 0"/>
@@ -30,7 +30,6 @@
         </geometry>
       </collision>
-      <self_collide>true</self_collide>
-    </link>
-    <link name="left_link1_1">
+    </link>
+    <link name="${prefix}left_link1_1">
       <inertial>
         <origin xyz="3.2842893861874216e-09 0.0339438363239903 0.004338426588372579" rpy="0 0 0"/>
@@ -51,7 +50,6 @@
         </geometry>
       </collision>
-      <self_collide>true</self_collide>
-    </link>
-    <link name="right_link1_1">
+    </link>
+    <link name="${prefix}right_link1_1">
       <inertial>
         <origin xyz="-3.2842893531192553e-09 -0.03394383632399016 0.004338426588372579" rpy="0 0 0"/>
@@ -72,7 +70,6 @@
         </geometry>
       </collision>
-      <self_collide>true</self_collide>
-    </link>
-    <link name="neck_link1_1">
+    </link>
+    <link name="${prefix}neck_link1_1">
       <inertial>
         <origin xyz="-0.00030973850909889926 -0.014644333953918068 0.03569874341148194" rpy="0 0 0"/>
@@ -93,7 +90,6 @@
         </geometry>
       </collision>
-      <self_collide>true</self_collide>
-    </link>
-    <link name="neck_link2_1">
+    </link>
+    <link name="${prefix}neck_link2_1">
       <inertial>
         <origin xyz="0.013634139305983414 0.0007303949446386359 0.035430103721878825" rpy="0 0 0"/>
@@ -114,7 +110,6 @@
         </geometry>
       </collision>
-      <self_collide>true</self_collide>
-    </link>
-    <link name="left_link2_1">
+    </link>
+    <link name="${prefix}left_link2_1">
       <inertial>
         <origin xyz="-0.02738813477340827 0.0003646764139110803 -0.06351763830886736" rpy="0 0 0"/>
@@ -135,7 +130,6 @@
         </geometry>
       </collision>
-      <self_collide>true</self_collide>
-    </link>
-    <link name="left_link3_1">
+    </link>
+    <link name="${prefix}left_link3_1">
       <inertial>
         <origin xyz="-1.2092751239928777e-08 1.2973242757841064e-09 -0.026072371405695793" rpy="0 0 0"/>
@@ -156,7 +150,6 @@
         </geometry>
       </collision>
-      <self_collide>true</self_collide>
-    </link>
-    <link name="left_link4_1">
+    </link>
+    <link name="${prefix}left_link4_1">
       <inertial>
         <origin xyz="-0.004070974019487877 -0.018903692607189798 -0.06334059246636403" rpy="0 0 0"/>
@@ -177,7 +170,6 @@
         </geometry>
       </collision>
-      <self_collide>true</self_collide>
-    </link>
-    <link name="left_link5_1">
+    </link>
+    <link name="${prefix}left_link5_1">
       <inertial>
         <origin xyz="2.8685271546600392e-08 1.2810758009962342e-09 -0.017987620476692334" rpy="0 0 0"/>
@@ -198,7 +190,6 @@
         </geometry>
       </collision>
-      <self_collide>true</self_collide>
-    </link>
-    <link name="left_link6_1">
+    </link>
+    <link name="${prefix}left_link6_1">
       <inertial>
         <origin xyz="0.00017312528224349425 -0.02085009010277386 -0.030500463697734653" rpy="0 0 0"/>
@@ -219,7 +210,6 @@
         </geometry>
       </collision>
-      <self_collide>true</self_collide>
-    </link>
-    <link name="left_link_gripper_1">
+    </link>
+    <link name="${prefix}left_link_gripper_1">
       <inertial>
         <origin xyz="-0.022004443717257835 0.018430761900261827 -0.031128994083327033" rpy="0 0 0"/>
@@ -240,7 +230,6 @@
         </geometry>
       </collision>
-      <self_collide>true</self_collide>
-    </link>
-    <link name="right_link2_1">
+    </link>
+    <link name="${prefix}right_link2_1">
       <inertial>
         <origin xyz="-0.02727565185538715 -0.00036463615065041033 -0.06351762777052061" rpy="0 0 0"/>
@@ -261,7 +250,6 @@
         </geometry>
       </collision>
-      <self_collide>true</self_collide>
-    </link>
-    <link name="right_link3_1">
+    </link>
+    <link name="${prefix}right_link3_1">
       <inertial>
         <origin xyz="-1.209275128617e-08 -1.2656755643547513e-09 -0.026072371405695682" rpy="0 0 0"/>
@@ -282,7 +270,6 @@
         </geometry>
       </collision>
-      <self_collide>true</self_collide>
-    </link>
-    <link name="right_link4_1">
+    </link>
+    <link name="${prefix}right_link4_1">
       <inertial>
         <origin xyz="-0.0040709740464307306 0.018876725019776414 -0.06334059246636403" rpy="0 0 0"/>
@@ -303,7 +290,6 @@
         </geometry>
       </collision>
-      <self_collide>true</self_collide>
-    </link>
-    <link name="right_link5_1">
+    </link>
+    <link name="${prefix}right_link5_1">
       <inertial>
         <origin xyz="2.8685270933538273e-08 -1.2819240391426234e-09 -0.01798762047669228" rpy="0 0 0"/>
@@ -324,7 +310,6 @@
         </geometry>
       </collision>
-      <self_collide>true</self_collide>
-    </link>
-    <link name="right_link6_1">
+    </link>
+    <link name="${prefix}right_link6_1">
       <inertial>
         <origin xyz="0.00017312522335896592 0.020213672315239545 -0.03049306440428448" rpy="0 0 0"/>
@@ -345,7 +330,6 @@
         </geometry>
       </collision>
-      <self_collide>true</self_collide>
-    </link>
-    <link name="right_link_gripper_1">
+    </link>
+    <link name="${prefix}right_link_gripper_1">
       <inertial>
         <origin xyz="-0.01899555242215849 -0.01843075902288205 -0.031128985762427674" rpy="0 0 0"/>
@@ -366,10 +350,9 @@
         </geometry>
       </collision>
-      <self_collide>true</self_collide>
     </link>
     <joint name="right_joint1" type="continuous">
       <origin xyz="0.00025 -0.1025 0.6155" rpy="0 0 0"/>
-      <parent link="base_link"/>
-      <child link="right_link1_1"/>
+      <parent link="${prefix}base_link"/>
+      <child link="${prefix}right_link1_1"/>
       <axis xyz="-0.0 -1.0 0.0"/>
       <limit velocity="4.8" effort="30" lower="${-pi*2.0}" upper="${pi*2.0}" />
@@ -378,6 +361,6 @@
     <joint name="right_joint2" type="continuous">
       <origin xyz="0.0245 -0.05 0.0" rpy="0 0 0"/>
-      <parent link="right_link1_1"/>
-      <child link="right_link2_1"/>
+      <parent link="${prefix}right_link1_1"/>
+      <child link="${prefix}right_link2_1"/>
       <axis xyz="-1.0 -0.0 0.0"/>
       <limit velocity="4.8" effort="30" lower="${-pi*2.0}" upper="${pi*2.0}" />
@@ -386,6 +369,6 @@
     <joint name="right_joint3" type="continuous">
       <origin xyz="-0.0245 0.0 -0.15775" rpy="0 0 0"/>
-      <parent link="right_link2_1"/>
-      <child link="right_link3_1"/>
+      <parent link="${prefix}right_link2_1"/>
+      <child link="${prefix}right_link3_1"/>
       <axis xyz="0.0 -0.0 -1.0"/>
       <limit velocity="4.8" effort="30" lower="${-pi*2.0}" upper="${pi*2.0}" />
@@ -394,6 +377,6 @@
     <joint name="right_joint4" type="continuous">
       <origin xyz="0.0 -0.019 -0.0315" rpy="0 0 0"/>
-      <parent link="right_link3_1"/>
-      <child link="right_link4_1"/>
+      <parent link="${prefix}right_link3_1"/>
+      <child link="${prefix}right_link4_1"/>
       <axis xyz="0.0 1.0 -0.0"/>
       <limit velocity="4.8" effort="30" lower="${-pi*2.0}" upper="${pi*2.0}" />
@@ -402,6 +385,6 @@
     <joint name="right_joint5" type="continuous">
       <origin xyz="0.0 0.019 -0.1401" rpy="0 0 0"/>
-      <parent link="right_link4_1"/>
-      <child link="right_link5_1"/>
+      <parent link="${prefix}right_link4_1"/>
+      <child link="${prefix}right_link5_1"/>
       <axis xyz="0.0 0.0 -1.0"/>
       <limit velocity="4.8" effort="30" lower="${-pi*2.0}" upper="${pi*2.0}" />
@@ -410,6 +393,6 @@
     <joint name="right_joint6" type="continuous">
       <origin xyz="0.0 -0.019 -0.0315" rpy="0 0 0"/>
-      <parent link="right_link5_1"/>
-      <child link="right_link6_1"/>
+      <parent link="${prefix}right_link5_1"/>
+      <child link="${prefix}right_link6_1"/>
       <axis xyz="0.0 1.0 0.0"/>
       <limit velocity="4.8" effort="30" lower="${-pi*2.0}" upper="${pi*2.0}" />
@@ -418,6 +401,6 @@
     <joint name="right_joint_gripper" type="continuous">
       <origin xyz="0.019 0.007 -0.0495" rpy="0 0 0"/>
-      <parent link="right_link6_1"/>
-      <child link="right_link_gripper_1"/>
+      <parent link="${prefix}right_link6_1"/>
+      <child link="${prefix}right_link_gripper_1"/>
       <axis xyz="1.0 -0.0 -0.0"/>
       <limit velocity="4.8" effort="30" lower="${-pi*2.0}" upper="${pi*2.0}" />
@@ -426,6 +409,6 @@
     <joint name="left_joint1" type="continuous">
       <origin xyz="-0.00025 0.1025 0.6155" rpy="0 0 0"/>
-      <parent link="base_link"/>
-      <child link="left_link1_1"/>
+      <parent link="${prefix}base_link"/>
+      <child link="${prefix}left_link1_1"/>
       <axis xyz="0.0 1.0 0.0"/>
       <limit velocity="4.8" effort="30" lower="${-pi*2.0}" upper="${pi*2.0}" />
@@ -434,6 +417,6 @@
     <joint name="left_joint2" type="continuous">
       <origin xyz="0.0245 0.05 0.0" rpy="0 0 0"/>
-      <parent link="left_link1_1"/>
-      <child link="left_link2_1"/>
+      <parent link="${prefix}left_link1_1"/>
+      <child link="${prefix}left_link2_1"/>
       <axis xyz="-1.0 -0.0 -0.0"/>
       <limit velocity="4.8" effort="30" lower="${-pi*2.0}" upper="${pi*2.0}" />
@@ -442,6 +425,6 @@
     <joint name="left_joint3" type="continuous">
       <origin xyz="-0.0245 0.0 -0.15775" rpy="0 0 0"/>
-      <parent link="left_link2_1"/>
-      <child link="left_link3_1"/>
+      <parent link="${prefix}left_link2_1"/>
+      <child link="${prefix}left_link3_1"/>
       <axis xyz="0.0 -0.0 -1.0"/>
       <limit velocity="4.8" effort="30" lower="${-pi*2.0}" upper="${pi*2.0}" />
@@ -450,6 +433,6 @@
     <joint name="left_joint4" type="continuous">
       <origin xyz="0.0 0.019 -0.0315" rpy="0 0 0"/>
-      <parent link="left_link3_1"/>
-      <child link="left_link4_1"/>
+      <parent link="${prefix}left_link3_1"/>
+      <child link="${prefix}left_link4_1"/>
       <axis xyz="-0.0 -1.0 0.0"/>
       <limit velocity="4.8" effort="30" lower="${-pi*2.0}" upper="${pi*2.0}" />
@@ -458,6 +441,6 @@
     <joint name="left_joint5" type="continuous">
       <origin xyz="0.0 -0.019 -0.1401" rpy="0 0 0"/>
-      <parent link="left_link4_1"/>
-      <child link="left_link5_1"/>
+      <parent link="${prefix}left_link4_1"/>
+      <child link="${prefix}left_link5_1"/>
       <axis xyz="0.0 0.0 -1.0"/>
       <limit velocity="4.8" effort="30" lower="${-pi*2.0}" upper="${pi*2.0}" />
@@ -466,6 +449,6 @@
     <joint name="left_joint6" type="continuous">
       <origin xyz="0.0 0.019 -0.0315" rpy="0 0 0"/>
-      <parent link="left_link5_1"/>
-      <child link="left_link6_1"/>
+      <parent link="${prefix}left_link5_1"/>
+      <child link="${prefix}left_link6_1"/>
       <axis xyz="-0.0 -1.0 -0.0"/>
       <limit velocity="4.8" effort="30" lower="${-pi*2.0}" upper="${pi*2.0}" />
@@ -474,6 +457,6 @@
     <joint name="left_joint_gripper" type="continuous">
       <origin xyz="0.019 -0.0086 -0.0495" rpy="0 0 0"/>
-      <parent link="left_link6_1"/>
-      <child link="left_link_gripper_1"/>
+      <parent link="${prefix}left_link6_1"/>
+      <child link="${prefix}left_link_gripper_1"/>
       <axis xyz="1.0 -0.0 -0.0"/>
       <limit velocity="4.8" effort="30" lower="${-pi*2.0}" upper="${pi*2.0}" />
@@ -482,6 +465,6 @@
     <joint name="neck_joint1" type="continuous">
       <origin xyz="0.00025 0.0194 0.6478" rpy="0 0 0"/>
-      <parent link="base_link"/>
-      <child link="neck_link1_1"/>
+      <parent link="${prefix}base_link"/>
+      <child link="${prefix}neck_link1_1"/>
       <axis xyz="0.0 1.0 -0.0"/>
       <limit velocity="4.8" effort="30" lower="${-pi*2.0}" upper="${pi*2.0}" />
@@ -490,6 +473,6 @@
     <joint name="neck_joint2" type="continuous">
       <origin xyz="0.0 -0.019 0.05975" rpy="0 0 0"/>
-      <parent link="neck_link1_1"/>
-      <child link="neck_link2_1"/>
+      <parent link="${prefix}neck_link1_1"/>
+      <child link="${prefix}neck_link2_1"/>
       <axis xyz="0.0 0.0 1.0"/>
       <limit velocity="4.8" effort="30" lower="${-pi*2.0}" upper="${pi*2.0}" />
@@ -497,5 +480,12 @@
     </joint>
     <!-- Contact sensors for collision detection -->
-    <gazebo reference="base_link">
+    <gazebo reference="${prefix}base_link">
+      <self_collide>true</self_collide>
+      <kp>1000000.0</kp>
+      <kd>100.0</kd>
+      <mu1>30.0</mu1>
+      <mu2>30.0</mu2>
+      <maxVel>1.0</maxVel>
+      <minDepth>0.001</minDepth>
       <sensor name="base_link_bumper" type="contact">
         <always_on>true</always_on>
@@ -509,5 +499,12 @@
       </sensor>
     </gazebo>
-    <gazebo reference="left_link1_1">
+    <gazebo reference="${prefix}left_link1_1">
+      <self_collide>true</self_collide>
+      <kp>1000000.0</kp>
+      <kd>100.0</kd>
+      <mu1>30.0</mu1>
+      <mu2>30.0</mu2>
+      <maxVel>1.0</maxVel>
+      <minDepth>0.001</minDepth>
       <sensor name="left_link1_1_bumper" type="contact">
         <always_on>true</always_on>
@@ -521,5 +518,12 @@
       </sensor>
     </gazebo>
-    <gazebo reference="right_link1_1">
+    <gazebo reference="${prefix}right_link1_1">
+      <self_collide>true</self_collide>
+      <kp>1000000.0</kp>
+      <kd>100.0</kd>
+      <mu1>30.0</mu1>
+      <mu2>30.0</mu2>
+      <maxVel>1.0</maxVel>
+      <minDepth>0.001</minDepth>
       <sensor name="right_link1_1_bumper" type="contact">
         <always_on>true</always_on>
@@ -533,5 +537,12 @@
       </sensor>
     </gazebo>
-    <gazebo reference="neck_link1_1">
+    <gazebo reference="${prefix}neck_link1_1">
+      <self_collide>true</self_collide>
+      <kp>1000000.0</kp>
+      <kd>100.0</kd>
+      <mu1>30.0</mu1>
+      <mu2>30.0</mu2>
+      <maxVel>1.0</maxVel>
+      <minDepth>0.001</minDepth>
       <sensor name="neck_link1_1_bumper" type="contact">
         <always_on>true</always_on>
@@ -545,5 +556,12 @@
       </sensor>
     </gazebo>
-    <gazebo reference="neck_link2_1">
+    <gazebo reference="${prefix}neck_link2_1">
+      <self_collide>true</self_collide>
+      <kp>1000000.0</kp>
+      <kd>100.0</kd>
+      <mu1>30.0</mu1>
+      <mu2>30.0</mu2>
+      <maxVel>1.0</maxVel>
+      <minDepth>0.001</minDepth>
       <sensor name="neck_link2_1_bumper" type="contact">
         <always_on>true</always_on>
@@ -557,5 +575,12 @@
       </sensor>
     </gazebo>
-    <gazebo reference="left_link2_1">
+    <gazebo reference="${prefix}left_link2_1">
+      <self_collide>true</self_collide>
+      <kp>1000000.0</kp>
+      <kd>100.0</kd>
+      <mu1>30.0</mu1>
+      <mu2>30.0</mu2>
+      <maxVel>1.0</maxVel>
+      <minDepth>0.001</minDepth>
       <sensor name="left_link2_1_bumper" type="contact">
         <always_on>true</always_on>
@@ -569,5 +594,12 @@
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