Commit message: 토픽 리스트에 띄움

File: avatar_description/gazebo/follower.gazebo.xacro (robot description, xacro)
@@ -57,4 +57,280 @@
     <xacro:SimpleTransmission trans="${prefix}trans15" joint="${prefix}neck_joint1" actuator="${prefix}actuator15" />
     <xacro:SimpleTransmission trans="${prefix}trans16" joint="${prefix}neck_joint2" actuator="${prefix}actuator16" />
+     <!-- Contact sensors for collision detection -->
+    <gazebo reference="${prefix}base_link">
+      <self_collide>true</self_collide>
+      <kp>1000000.0</kp>
+      <kd>100.0</kd>
+      <mu1>30.0</mu1>
+      <mu2>30.0</mu2>
+      <maxVel>1.0</maxVel>
+      <minDepth>0.001</minDepth>
+      <sensor name="base_link_bumper" type="contact">
+        <always_on>true</always_on>
+        <update_rate>50.0</update_rate>
+        <contact>
+          <collision>${prefix}base_link_collision</collision>
+        </contact>
+      </sensor>
+      <plugin filename="libignition-gazebo-touchplugin-system.so"
+                name="ignition::gazebo::systems::TouchPlugin">
+        </plugin>
+    </gazebo>
+    <gazebo reference="${prefix}left_link1_1">
+      <self_collide>true</self_collide>
+      <kp>1000000.0</kp>
+      <kd>100.0</kd>
+      <mu1>30.0</mu1>
+      <mu2>30.0</mu2>
+      <maxVel>1.0</maxVel>
+      <minDepth>0.001</minDepth>
+      <sensor name="left_link1_1_bumper" type="contact">
+        <always_on>true</always_on>
+        <update_rate>50.0</update_rate>
+        <contact>
+          <collision>${prefix}left_link1_1_collision</collision>
+        </contact>
+      </sensor>
+    </gazebo>
+    <gazebo reference="${prefix}right_link1_1">
+      <self_collide>true</self_collide>
+      <kp>1000000.0</kp>
+      <kd>100.0</kd>
+      <mu1>30.0</mu1>
+      <mu2>30.0</mu2>
+      <maxVel>1.0</maxVel>
+      <minDepth>0.001</minDepth>
+      <sensor name="right_link1_1_bumper" type="contact">
+        <always_on>true</always_on>
+        <update_rate>50.0</update_rate>
+        <contact>
+          <collision>${prefix}right_link1_1_collision</collision>
+        </contact>
+      </sensor>
+    </gazebo>
+    <gazebo reference="${prefix}neck_link1_1">
+      <self_collide>true</self_collide>
+      <kp>1000000.0</kp>
+      <kd>100.0</kd>
+      <mu1>30.0</mu1>
+      <mu2>30.0</mu2>
+      <maxVel>1.0</maxVel>
+      <minDepth>0.001</minDepth>
+      <sensor name="neck_link1_1_bumper" type="contact">
+        <always_on>true</always_on>
+        <update_rate>50.0</update_rate>
+        <contact>
+          <collision>${prefix}neck_link1_1_collision</collision>
+        </contact>
+      </sensor>
+    </gazebo>
+    <gazebo reference="${prefix}neck_link2_1">
+      <self_collide>true</self_collide>
+      <kp>1000000.0</kp>
+      <kd>100.0</kd>
+      <mu1>30.0</mu1>
+      <mu2>30.0</mu2>
+      <maxVel>1.0</maxVel>
+      <minDepth>0.001</minDepth>
+      <sensor name="neck_link2_1_bumper" type="contact">
+        <always_on>true</always_on>
+        <update_rate>50.0</update_rate>
+        <contact>
+          <collision>${prefix}neck_link2_1_collision</collision>
+        </contact>
+      </sensor>
+    </gazebo>
+    <gazebo reference="${prefix}left_link2_1">
+      <self_collide>true</self_collide>
+      <kp>1000000.0</kp>
+      <kd>100.0</kd>
+      <mu1>30.0</mu1>
+      <mu2>30.0</mu2>
+      <maxVel>1.0</maxVel>
+      <minDepth>0.001</minDepth>
+      <sensor name="left_link2_1_bumper" type="contact">
+        <always_on>true</always_on>
+        <update_rate>50.0</update_rate>
+        <contact>
+          <collision>${prefix}left_link2_1_collision</collision>
+        </contact>
+      </sensor>
+    </gazebo>
+    <gazebo reference="${prefix}left_link3_1">
+      <self_collide>true</self_collide>
+      <kp>1000000.0</kp>
+      <kd>100.0</kd>
+      <mu1>30.0</mu1>
+      <mu2>30.0</mu2>
+      <maxVel>1.0</maxVel>
+      <minDepth>0.001</minDepth>
+      <sensor name="left_link3_1_bumper" type="contact">
+        <always_on>true</always_on>
+        <update_rate>50.0</update_rate>
+        <contact>
+          <collision>${prefix}left_link3_1_collision</collision>
+        </contact>
+      </sensor>
+    </gazebo>
+    <gazebo reference="${prefix}left_link4_1">
+      <self_collide>true</self_collide>
+      <kp>1000000.0</kp>
+      <kd>100.0</kd>
+      <mu1>30.0</mu1>
+      <mu2>30.0</mu2>
+      <maxVel>1.0</maxVel>
+      <minDepth>0.001</minDepth>
+      <sensor name="left_link4_1_bumper" type="contact">
+        <always_on>true</always_on>
+        <update_rate>50.0</update_rate>
+        <contact>
+          <collision>${prefix}left_link4_1_collision</collision>
+        </contact>
+      </sensor>
+    </gazebo>
+    <gazebo reference="${prefix}left_link5_1">
+      <self_collide>true</self_collide>
+      <kp>1000000.0</kp>
+      <kd>100.0</kd>
+      <mu1>30.0</mu1>
+      <mu2>30.0</mu2>
+      <maxVel>1.0</maxVel>
+      <minDepth>0.001</minDepth>
+      <sensor name="left_link5_1_bumper" type="contact">
+        <always_on>true</always_on>
+        <update_rate>50.0</update_rate>
+        <contact>
+          <collision>${prefix}left_link5_1_collision</collision>
+        </contact>
+      </sensor>
+    </gazebo>
+    <gazebo reference="${prefix}left_link6_1">
+      <self_collide>true</self_collide>
+      <kp>1000000.0</kp>
+      <kd>100.0</kd>
+      <mu1>30.0</mu1>
+      <mu2>30.0</mu2>
+      <maxVel>1.0</maxVel>
+      <minDepth>0.001</minDepth>
+      <sensor name="left_link6_1_bumper" type="contact">
+        <always_on>true</always_on>
+        <update_rate>50.0</update_rate>
+        <contact>
+          <collision>${prefix}left_link6_1_collision</collision>
+        </contact>
+      </sensor>
+    </gazebo>
+    <gazebo reference="${prefix}left_link_gripper_1">
+      <self_collide>true</self_collide>
+      <kp>1000000.0</kp>
+      <kd>100.0</kd>
+      <mu1>30.0</mu1>
+      <mu2>30.0</mu2>
+      <maxVel>1.0</maxVel>
+      <minDepth>0.001</minDepth>
+      <sensor name="left_gripper_bumper" type="contact">
+        <always_on>true</always_on>
+        <update_rate>50.0</update_rate>
+        <contact>
+          <collision>${prefix}left_link_gripper_1_collision</collision>
+        </contact>
+      </sensor>
+    </gazebo>
+    <gazebo reference="${prefix}right_link2_1">
+      <self_collide>true</self_collide>
+      <kp>1000000.0</kp>
+      <kd>100.0</kd>
+      <mu1>30.0</mu1>
+      <mu2>30.0</mu2>
+      <maxVel>1.0</maxVel>
+      <minDepth>0.001</minDepth>
+      <sensor name="right_link2_1_bumper" type="contact">
+        <always_on>true</always_on>
+        <update_rate>50.0</update_rate>
+        <contact>
+          <collision>${prefix}right_link2_1_collision</collision>
+        </contact>
+      </sensor>
+    </gazebo>
+    <gazebo reference="${prefix}right_link3_1">
+      <self_collide>true</self_collide>
+      <kp>1000000.0</kp>
+      <kd>100.0</kd>
+      <mu1>30.0</mu1>
+      <mu2>30.0</mu2>
+      <maxVel>1.0</maxVel>
+      <minDepth>0.001</minDepth>
+      <sensor name="right_link3_1_bumper" type="contact">
+        <always_on>true</always_on>
+        <update_rate>50.0</update_rate>
+        <contact>
+          <collision>${prefix}right_link3_1_collision</collision>
+        </contact>
+      </sensor>
+    </gazebo>
+    <gazebo reference="${prefix}right_link4_1">
+      <self_collide>true</self_collide>
+      <kp>1000000.0</kp>
+      <kd>100.0</kd>
+      <mu1>30.0</mu1>
+      <mu2>30.0</mu2>
+      <maxVel>1.0</maxVel>
+      <minDepth>0.001</minDepth>
+      <sensor name="right_link4_1_bumper" type="contact">
+        <always_on>true</always_on>
+        <update_rate>50.0</update_rate>
+        <contact>
+          <collision>${prefix}right_link4_1_collision</collision>
+        </contact>
+      </sensor>
+    </gazebo>
+    <gazebo reference="${prefix}right_link5_1">
+      <self_collide>true</self_collide>
+      <kp>1000000.0</kp>
+      <kd>100.0</kd>
+      <mu1>30.0</mu1>
+      <mu2>30.0</mu2>
+      <maxVel>1.0</maxVel>
+      <minDepth>0.001</minDepth>
+      <sensor name="right_link5_1_bumper" type="contact">
+        <always_on>true</always_on>
+        <update_rate>50.0</update_rate>
+        <contact>
+          <collision>${prefix}right_link5_1_collision</collision>
+        </contact>
+      </sensor>
+    </gazebo>
+    <gazebo reference="${prefix}right_link6_1">
+      <self_collide>true</self_collide>
+      <kp>1000000.0</kp>
+      <kd>100.0</kd>
+      <mu1>30.0</mu1>
+      <mu2>30.0</mu2>
+      <maxVel>1.0</maxVel>
+      <minDepth>0.001</minDepth>
+      <sensor name="right_link6_1_bumper" type="contact">
+        <always_on>true</always_on>
+        <update_rate>50.0</update_rate>
+        <contact>
+          <collision>${prefix}right_link6_1_collision</collision>
+        </contact>
+      </sensor>
+    </gazebo>
+    <gazebo reference="${prefix}right_link_gripper_1">
+      <self_collide>true</self_collide>
+      <kp>1000000.0</kp>
+      <kd>100.0</kd>
+      <mu1>30.0</mu1>
+      <mu2>30.0</mu2>
+      <maxVel>1.0</maxVel>
+      <minDepth>0.001</minDepth>
+      <sensor name="right_gripper_bumper" type="contact">
+        <always_on>true</always_on>
+        <update_rate>50.0</update_rate>
+        <contact>
+          <collision>${prefix}right_link_gripper_1_collision</collision>
+        </contact>
+      </sensor>
+    </gazebo>
   </xacro:macro>
 </robot>
