Commit message: 토픽 리스트에 띄움

File: avatar_description/urdf/follower/follower_arm.urdf.xacro (robot description, xacro)
@@ -24,5 +24,5 @@
         <material name="dark_gray"/>
       </visual>
-      <collision name="${prefix}base_link_collision">
+      <collision>
         <origin xyz="0 0 0" rpy="0 0 0"/>
         <geometry>
@@ -44,5 +44,5 @@
         <material name="dark_gray"/>
       </visual>
-      <collision name="${prefix}left_link1_1_collision">
+       <collision>
         <origin xyz="0.00025 -0.1025 -0.6155" rpy="0 0 0"/>
         <geometry>
@@ -64,5 +64,5 @@
         <material name="dark_gray"/>
       </visual>
-      <collision name="${prefix}right_link1_1_collision">
+       <collision>
         <origin xyz="-0.00025 0.1025 -0.6155" rpy="0 0 0"/>
         <geometry>
@@ -84,5 +84,5 @@
         <material name="dark_gray"/>
       </visual>
-      <collision name="${prefix}neck_link1_1_collision">
+       <collision>
         <origin xyz="-0.00025 -0.0194 -0.6478" rpy="0 0 0"/>
         <geometry>
@@ -104,5 +104,5 @@
         <material name="white"/>
       </visual>
-      <collision name="${prefix}neck_link2_1_collision">
+       <collision>
         <origin xyz="-0.00025 -0.0004 -0.70755" rpy="0 0 0"/>
         <geometry>
@@ -124,5 +124,5 @@
         <material name="dark_gray"/>
       </visual>
-      <collision name="${prefix}left_link2_1_collision">
+       <collision>
         <origin xyz="-0.02425 -0.1525 -0.6155" rpy="0 0 0"/>
         <geometry>
@@ -144,5 +144,5 @@
         <material name="dark_gray"/>
       </visual>
-      <collision name="${prefix}left_link3_1_collision">
+       <collision>
         <origin xyz="0.00025 -0.1525 -0.45775" rpy="0 0 0"/>
         <geometry>
@@ -164,5 +164,5 @@
         <material name="dark_gray"/>
       </visual>
-      <collision name="${prefix}left_link4_1_collision">
+       <collision>
         <origin xyz="0.00025 -0.1715 -0.42625" rpy="0 0 0"/>
         <geometry>
@@ -184,5 +184,5 @@
         <material name="dark_gray"/>
       </visual>
-      <collision name="${prefix}left_link5_1_collision">
+       <collision>
         <origin xyz="0.00025 -0.1525 -0.28615" rpy="0 0 0"/>
         <geometry>
@@ -204,5 +204,5 @@
         <material name="dark_gray"/>
       </visual>
-      <collision name="${prefix}left_link6_1_collision">
+       <collision>
         <origin xyz="0.00025 -0.1715 -0.25465" rpy="0 0 0"/>
         <geometry>
@@ -224,5 +224,5 @@
         <material name="dark_gray"/>
       </visual>
-      <collision name="${prefix}left_link_gripper_1_collision">
+       <collision>
         <origin xyz="-0.01875 -0.1629 -0.20515" rpy="0 0 0"/>
         <geometry>
@@ -244,5 +244,5 @@
         <material name="dark_gray"/>
       </visual>
-      <collision name="${prefix}right_link2_1_collision">
+       <collision>
         <origin xyz="-0.02475 0.1525 -0.6155" rpy="0 0 0"/>
         <geometry>
@@ -264,5 +264,5 @@
         <material name="dark_gray"/>
       </visual>
-      <collision name="${prefix}right_link3_1_collision">
+       <collision>
         <origin xyz="-0.00025 0.1525 -0.45775" rpy="0 0 0"/>
         <geometry>
@@ -284,5 +284,5 @@
         <material name="dark_gray"/>
       </visual>
-      <collision name="${prefix}right_link4_1_collision">
+       <collision>
         <origin xyz="-0.00025 0.1715 -0.42625" rpy="0 0 0"/>
         <geometry>
@@ -304,5 +304,5 @@
         <material name="dark_gray"/>
       </visual>
-      <collision name="${prefix}right_link5_1_collision">
+       <collision>
         <origin xyz="-0.00025 0.1525 -0.28615" rpy="0 0 0"/>
         <geometry>
@@ -324,5 +324,5 @@
         <material name="dark_gray"/>
       </visual>
-      <collision name="${prefix}right_link6_1_collision">
+       <collision>
         <origin xyz="-0.00025 0.1715 -0.25465" rpy="0 0 0"/>
         <geometry>
@@ -344,5 +344,5 @@
         <material name="dark_gray"/>
       </visual>
-      <collision name="${prefix}right_link_gripper_1_collision">
+       <collision>
         <origin xyz="-0.01925 0.1645 -0.20515" rpy="0 0 0"/>
         <geometry>
@@ -479,328 +479,4 @@
       <dynamics damping="0.1" />
     </joint>
-    <!-- Contact sensors for collision detection -->
-    <gazebo reference="${prefix}base_link">
-      <self_collide>true</self_collide>
-      <kp>1000000.0</kp>
-      <kd>100.0</kd>
-      <mu1>30.0</mu1>
-      <mu2>30.0</mu2>
-      <maxVel>1.0</maxVel>
-      <minDepth>0.001</minDepth>
-      <sensor name="base_link_bumper" type="contact">
-        <always_on>true</always_on>
-        <update_rate>50.0</update_rate>
-        <contact>
-          <collision>${prefix}base_link_collision</collision>
-        </contact>
-        <plugin filename="libignition-gazebo-contact-system.so"
-                name="ignition::gazebo::systems::Contact">
-        </plugin>
-      </sensor>
-    </gazebo>
-    <gazebo reference="${prefix}left_link1_1">
-      <self_collide>true</self_collide>
-      <kp>1000000.0</kp>
-      <kd>100.0</kd>
-      <mu1>30.0</mu1>
-      <mu2>30.0</mu2>
-      <maxVel>1.0</maxVel>
-      <minDepth>0.001</minDepth>
-      <sensor name="left_link1_1_bumper" type="contact">
-        <always_on>true</always_on>
-        <update_rate>50.0</update_rate>
-        <contact>
-          <collision>${prefix}left_link1_1_collision</collision>
-        </contact>
-        <plugin filename="libignition-gazebo-contact-system.so"
-                name="ignition::gazebo::systems::Contact">
-        </plugin>
-      </sensor>
-    </gazebo>
-    <gazebo reference="${prefix}right_link1_1">
-      <self_collide>true</self_collide>
-      <kp>1000000.0</kp>
-      <kd>100.0</kd>
-      <mu1>30.0</mu1>
-      <mu2>30.0</mu2>
-      <maxVel>1.0</maxVel>
-      <minDepth>0.001</minDepth>
-      <sensor name="right_link1_1_bumper" type="contact">
-        <always_on>true</always_on>
-        <update_rate>50.0</update_rate>
-        <contact>
-          <collision>${prefix}right_link1_1_collision</collision>
-        </contact>
-        <plugin filename="libignition-gazebo-contact-system.so"
-                name="ignition::gazebo::systems::Contact">
-        </plugin>
-      </sensor>
-    </gazebo>
-    <gazebo reference="${prefix}neck_link1_1">
-      <self_collide>true</self_collide>
-      <kp>1000000.0</kp>
-      <kd>100.0</kd>
-      <mu1>30.0</mu1>
-      <mu2>30.0</mu2>
-      <maxVel>1.0</maxVel>
-      <minDepth>0.001</minDepth>
-      <sensor name="neck_link1_1_bumper" type="contact">
-        <always_on>true</always_on>
-        <update_rate>50.0</update_rate>
-        <contact>
-          <collision>${prefix}neck_link1_1_collision</collision>
-        </contact>
-        <plugin filename="libignition-gazebo-contact-system.so"
-                name="ignition::gazebo::systems::Contact">
-        </plugin>
-      </sensor>
-    </gazebo>
-    <gazebo reference="${prefix}neck_link2_1">
-      <self_collide>true</self_collide>
-      <kp>1000000.0</kp>
-      <kd>100.0</kd>
-      <mu1>30.0</mu1>
-      <mu2>30.0</mu2>
-      <maxVel>1.0</maxVel>
-      <minDepth>0.001</minDepth>
-      <sensor name="neck_link2_1_bumper" type="contact">
-        <always_on>true</always_on>
-        <update_rate>50.0</update_rate>
-        <contact>
-          <collision>${prefix}neck_link2_1_collision</collision>
-        </contact>
-        <plugin filename="libignition-gazebo-contact-system.so"
-                name="ignition::gazebo::systems::Contact">
-        </plugin>
-      </sensor>
-    </gazebo>
-    <gazebo reference="${prefix}left_link2_1">
-      <self_collide>true</self_collide>
-      <kp>1000000.0</kp>
-      <kd>100.0</kd>
-      <mu1>30.0</mu1>
-      <mu2>30.0</mu2>
-      <maxVel>1.0</maxVel>
-      <minDepth>0.001</minDepth>
-      <sensor name="left_link2_1_bumper" type="contact">
-        <always_on>true</always_on>
-        <update_rate>50.0</update_rate>
-        <contact>
-          <collision>${prefix}left_link2_1_collision</collision>
-        </contact>
-        <plugin filename="libignition-gazebo-contact-system.so"
-                name="ignition::gazebo::systems::Contact">
-        </plugin>
-      </sensor>
-    </gazebo>
-    <gazebo reference="${prefix}left_link3_1">
-      <self_collide>true</self_collide>
-      <kp>1000000.0</kp>
-      <kd>100.0</kd>
-      <mu1>30.0</mu1>
-      <mu2>30.0</mu2>
-      <maxVel>1.0</maxVel>
-      <minDepth>0.001</minDepth>
-      <sensor name="left_link3_1_bumper" type="contact">
-        <always_on>true</always_on>
-        <update_rate>50.0</update_rate>
-        <contact>
-          <collision>${prefix}left_link3_1_collision</collision>
-        </contact>
-        <plugin filename="libignition-gazebo-contact-system.so"
-                name="ignition::gazebo::systems::Contact">
-        </plugin>
-      </sensor>
-    </gazebo>
-    <gazebo reference="${prefix}left_link4_1">
-      <self_collide>true</self_collide>
-      <kp>1000000.0</kp>
-      <kd>100.0</kd>
-      <mu1>30.0</mu1>
-      <mu2>30.0</mu2>
-      <maxVel>1.0</maxVel>
-      <minDepth>0.001</minDepth>
-      <sensor name="left_link4_1_bumper" type="contact">
-        <always_on>true</always_on>
-        <update_rate>50.0</update_rate>
-        <contact>
-          <collision>${prefix}left_link4_1_collision</collision>
-        </contact>
-        <plugin filename="libignition-gazebo-contact-system.so"
-                name="ignition::gazebo::systems::Contact">
-        </plugin>
-      </sensor>
-    </gazebo>
-    <gazebo reference="${prefix}left_link5_1">
-      <self_collide>true</self_collide>
-      <kp>1000000.0</kp>
-      <kd>100.0</kd>
-      <mu1>30.0</mu1>
-      <mu2>30.0</mu2>
-      <maxVel>1.0</maxVel>
-      <minDepth>0.001</minDepth>
-      <sensor name="left_link5_1_bumper" type="contact">
-        <always_on>true</always_on>
-        <update_rate>50.0</update_rate>
-        <contact>
-          <collision>${prefix}left_link5_1_collision</collision>
-        </contact>
-        <plugin filename="libignition-gazebo-contact-system.so"
-                name="ignition::gazebo::systems::Contact">
-        </plugin>
-      </sensor>
-    </gazebo>
-    <gazebo reference="${prefix}left_link6_1">
-      <self_collide>true</self_collide>
-      <kp>1000000.0</kp>
-      <kd>100.0</kd>
-      <mu1>30.0</mu1>
-      <mu2>30.0</mu2>
-      <maxVel>1.0</maxVel>
-      <minDepth>0.001</minDepth>
-      <sensor name="left_link6_1_bumper" type="contact">
-        <always_on>true</always_on>
-        <update_rate>50.0</update_rate>
-        <contact>
-          <collision>${prefix}left_link6_1_collision</collision>
-        </contact>
-        <plugin filename="libignition-gazebo-contact-system.so"
-                name="ignition::gazebo::systems::Contact">
-        </plugin>
-      </sensor>
-    </gazebo>
-    <gazebo reference="${prefix}left_link_gripper_1">
-      <self_collide>true</self_collide>
-      <kp>1000000.0</kp>
-      <kd>100.0</kd>
-      <mu1>30.0</mu1>
-      <mu2>30.0</mu2>
-      <maxVel>1.0</maxVel>
-      <minDepth>0.001</minDepth>
-      <sensor name="left_gripper_bumper" type="contact">
-        <always_on>true</always_on>
-        <update_rate>50.0</update_rate>
-        <contact>
-          <collision>${prefix}left_link_gripper_1_collision</collision>
-        </contact>
-        <plugin filename="libignition-gazebo-contact-system.so"
-                name="ignition::gazebo::systems::Contact">
-        </plugin>
-      </sensor>
-    </gazebo>
-    <gazebo reference="${prefix}right_link2_1">
-      <self_collide>true</self_collide>
-      <kp>1000000.0</kp>
-      <kd>100.0</kd>
-      <mu1>30.0</mu1>
-      <mu2>30.0</mu2>
-      <maxVel>1.0</maxVel>
-      <minDepth>0.001</minDepth>
-      <sensor name="right_link2_1_bumper" type="contact">
-        <always_on>true</always_on>
-        <update_rate>50.0</update_rate>
-        <contact>
-          <collision>${prefix}right_link2_1_collision</collision>
-        </contact>
-        <plugin filename="libignition-gazebo-contact-system.so"
-                name="ignition::gazebo::systems::Contact">
-        </plugin>
-      </sensor>
-    </gazebo>
-    <gazebo reference="${prefix}right_link3_1">
-      <self_collide>true</self_collide>
-      <kp>1000000.0</kp>
-      <kd>100.0</kd>
-      <mu1>30.0</mu1>
-      <mu2>30.0</mu2>
-      <maxVel>1.0</maxVel>
-      <minDepth>0.001</minDepth>
-      <sensor name="right_link3_1_bumper" type="contact">
-        <always_on>true</always_on>
-        <update_rate>50.0</update_rate>
-        <contact>
-          <collision>${prefix}right_link3_1_collision</collision>
-        </contact>
-        <plugin filename="libignition-gazebo-contact-system.so"
-                name="ignition::gazebo::systems::Contact">
-        </plugin>
-      </sensor>
-    </gazebo>
-    <gazebo reference="${prefix}right_link4_1">
-      <self_collide>true</self_collide>
-      <kp>1000000.0</kp>
-      <kd>100.0</kd>
-      <mu1>30.0</mu1>
-      <mu2>30.0</mu2>
-      <maxVel>1.0</maxVel>
-      <minDepth>0.001</minDepth>
-      <sensor name="right_link4_1_bumper" type="contact">
-        <always_on>true</always_on>
-        <update_rate>50.0</update_rate>
-        <contact>
-          <collision>${prefix}right_link4_1_collision</collision>
-        </contact>
-        <plugin filename="libignition-gazebo-contact-system.so"
-                name="ignition::gazebo::systems::Contact">
-        </plugin>
-      </sensor>
-    </gazebo>
-    <gazebo reference="${prefix}right_link5_1">
-      <self_collide>true</self_collide>
-      <kp>1000000.0</kp>
-      <kd>100.0</kd>
-      <mu1>30.0</mu1>
-      <mu2>30.0</mu2>
-      <maxVel>1.0</maxVel>
-      <minDepth>0.001</minDepth>
-      <sensor name="right_link5_1_bumper" type="contact">
-        <always_on>true</always_on>
-        <update_rate>50.0</update_rate>
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