Commit message: 가제보, 콜리션 업데이트 (콜리션은 아직 안됨)

File: avatar_description/ros2_control/follower.ros2_control.xacro (robot description, xacro)
@@ -198,6 +198,4 @@
           <param name="Min Position Limit">1024</param>
           <param name="Max Position Limit">3140</param>
-          <param name="Min Position Limit">830</param>
-          <param name="Max Position Limit">3129</param>
           <param name="Position P Gain">1000</param>
           <param name="Position I Gain">0</param>
@@ -217,6 +215,4 @@
           <param name="Min Position Limit">1024</param>
           <param name="Max Position Limit">3140</param>
-          <param name="Min Position Limit">830</param>
-          <param name="Max Position Limit">3129</param>
           <param name="Position P Gain">1000</param>
           <param name="Position I Gain">0</param>
@@ -236,6 +232,4 @@
           <param name="Min Position Limit">1024</param>
           <param name="Max Position Limit">3140</param>
-          <param name="Min Position Limit">830</param>
-          <param name="Max Position Limit">3129</param>
           <param name="Position P Gain">1000</param>
           <param name="Position I Gain">0</param>
@@ -255,6 +249,4 @@
           <param name="Min Position Limit">1024</param>
           <param name="Max Position Limit">3140</param>
-          <param name="Min Position Limit">830</param>
-          <param name="Max Position Limit">3129</param>
           <param name="Position P Gain">1000</param>
           <param name="Position I Gain">0</param>
@@ -274,6 +266,4 @@
           <param name="Min Position Limit">1024</param>
           <param name="Max Position Limit">3140</param>
-          <param name="Min Position Limit">830</param>
-          <param name="Max Position Limit">3129</param>
           <param name="Position P Gain">1000</param>
           <param name="Position I Gain">0</param>
@@ -293,6 +283,4 @@
           <param name="Min Position Limit">1024</param>
           <param name="Max Position Limit">3140</param>
-          <param name="Min Position Limit">830</param>
-          <param name="Max Position Limit">3129</param>
           <param name="Position P Gain">1000</param>
           <param name="Position I Gain">0</param>
@@ -312,6 +300,4 @@
           <param name="Min Position Limit">1024</param>
           <param name="Max Position Limit">3140</param>
-          <param name="Min Position Limit">830</param>
-          <param name="Max Position Limit">3129</param>
           <param name="Position P Gain">1000</param>
           <param name="Position I Gain">0</param>
@@ -331,6 +317,4 @@
           <param name="Min Position Limit">1024</param>
           <param name="Max Position Limit">3140</param>
-          <param name="Min Position Limit">830</param>
-          <param name="Max Position Limit">3129</param>
           <param name="Position P Gain">1000</param>
           <param name="Position I Gain">0</param>
@@ -350,6 +334,4 @@
           <param name="Min Position Limit">1024</param>
           <param name="Max Position Limit">3140</param>
-          <param name="Min Position Limit">830</param>
-          <param name="Max Position Limit">3129</param>
           <param name="Position P Gain">1000</param>
           <param name="Position I Gain">0</param>
@@ -369,6 +351,4 @@
           <param name="Min Position Limit">1024</param>
           <param name="Max Position Limit">3140</param>
-          <param name="Min Position Limit">830</param>
-          <param name="Max Position Limit">3129</param>
           <param name="Position P Gain">1000</param>
           <param name="Position I Gain">0</param>
@@ -388,6 +368,4 @@
           <param name="Min Position Limit">1024</param>
           <param name="Max Position Limit">3140</param>
-          <param name="Min Position Limit">830</param>
-          <param name="Max Position Limit">3129</param>
           <param name="Position P Gain">1000</param>
           <param name="Position I Gain">0</param>
@@ -407,6 +385,4 @@
           <param name="Min Position Limit">1024</param>
           <param name="Max Position Limit">3140</param>
-          <param name="Min Position Limit">830</param>
-          <param name="Max Position Limit">3129</param>
           <param name="Position P Gain">1000</param>
           <param name="Position I Gain">0</param>
@@ -426,6 +402,4 @@
           <param name="Min Position Limit">1024</param>
           <param name="Max Position Limit">3140</param>
-          <param name="Min Position Limit">830</param>
-          <param name="Max Position Limit">3129</param>
           <param name="Position P Gain">1000</param>
           <param name="Position I Gain">0</param>
@@ -445,6 +419,4 @@
           <param name="Min Position Limit">1024</param>
           <param name="Max Position Limit">3140</param>
-          <param name="Min Position Limit">830</param>
-          <param name="Max Position Limit">3129</param>
           <param name="Position P Gain">1000</param>
           <param name="Position I Gain">0</param>
@@ -464,6 +436,4 @@
           <param name="Min Position Limit">1024</param>
           <param name="Max Position Limit">3140</param>
-          <param name="Min Position Limit">830</param>
-          <param name="Max Position Limit">3129</param>
           <param name="Position P Gain">1000</param>
           <param name="Position I Gain">0</param>

File: avatar_description/urdf/follower/follower_arm.urdf.xacro (robot description, xacro)
@@ -363,5 +363,5 @@
       <parent link="${prefix}right_link1_1"/>
       <child link="${prefix}right_link2_1"/>
-      <axis xyz="-1.0 -0.0 0.0"/>
+      <axis xyz="1.0 -0.0 0.0"/>
       <limit velocity="4.8" effort="30" lower="${-pi*2.0}" upper="${pi*2.0}" />
       <dynamics damping="0.1" />
@@ -379,5 +379,5 @@
       <parent link="${prefix}right_link3_1"/>
       <child link="${prefix}right_link4_1"/>
-      <axis xyz="0.0 1.0 -0.0"/>
+      <axis xyz="0.0 -1.0 -0.0"/>
       <limit velocity="4.8" effort="30" lower="${-pi*2.0}" upper="${pi*2.0}" />
       <dynamics damping="0.1" />
@@ -395,5 +395,5 @@
       <parent link="${prefix}right_link5_1"/>
       <child link="${prefix}right_link6_1"/>
-      <axis xyz="0.0 1.0 0.0"/>
+      <axis xyz="0.0 -1.0 0.0"/>
       <limit velocity="4.8" effort="30" lower="${-pi*2.0}" upper="${pi*2.0}" />
       <dynamics damping="0.1" />
@@ -419,5 +419,5 @@
       <parent link="${prefix}left_link1_1"/>
       <child link="${prefix}left_link2_1"/>
-      <axis xyz="-1.0 -0.0 -0.0"/>
+      <axis xyz="1.0 -0.0 -0.0"/>
       <limit velocity="4.8" effort="30" lower="${-pi*2.0}" upper="${pi*2.0}" />
       <dynamics damping="0.1" />
@@ -435,5 +435,5 @@
       <parent link="${prefix}left_link3_1"/>
       <child link="${prefix}left_link4_1"/>
-      <axis xyz="-0.0 -1.0 0.0"/>
+      <axis xyz="-0.0 1.0 0.0"/>
       <limit velocity="4.8" effort="30" lower="${-pi*2.0}" upper="${pi*2.0}" />
       <dynamics damping="0.1" />
@@ -451,5 +451,5 @@
       <parent link="${prefix}left_link5_1"/>
       <child link="${prefix}left_link6_1"/>
-      <axis xyz="-0.0 -1.0 -0.0"/>
+      <axis xyz="-0.0 1.0 -0.0"/>
       <limit velocity="4.8" effort="30" lower="${-pi*2.0}" upper="${pi*2.0}" />
       <dynamics damping="0.1" />

Commit message: 가제보 각도 수정

File: avatar_description/ros2_control/follower.ros2_control.xacro (robot description, xacro)
@@ -283,5 +283,5 @@
           <param name="Min Position Limit">2048</param>
           <param name="Max Position Limit">3320</param>
-          <param name="Current Limit">200</param>
+          <param name="Current Limit">100</param>
           <param name="Position P Gain">1000</param>
           <param name="Position I Gain">0</param>
@@ -367,5 +367,5 @@
           <param name="Operating Mode">3</param>
           <param name="Return Delay Time">0</param>
-          <param name="Min Position Limit">2048</param>
+          <param name="Min Position Limit">1024</param>
           <param name="Max Position Limit">3072</param>
           <param name="Position P Gain">1000</param>
@@ -404,5 +404,5 @@
           <param name="Min Position Limit">776</param>
           <param name="Max Position Limit">2048</param>
-          <param name="Current Limit">200</param>
+          <param name="Current Limit">100</param>
           <param name="Position P Gain">1000</param>
           <param name="Position I Gain">0</param>

File: avatar_description/urdf/follower/follower_arm.urdf.xacro (robot description, xacro)
@@ -380,5 +380,5 @@
       <child link="${prefix}right_link4_1"/>
       <axis xyz="0.0 -1.0 -0.0"/>
-      <limit velocity="4.8" effort="30" lower="${-pi*0.389}" upper="${pi*0.389}" />
+      <limit velocity="4.8" effort="30" lower="${-pi*0.5}" upper="${pi*0.5}" />
       <dynamics damping="0.1" />
     </joint>
@@ -436,5 +436,5 @@
       <child link="${prefix}left_link4_1"/>
       <axis xyz="-0.0 1.0 0.0"/>
-      <limit velocity="4.8" effort="30" lower="${-pi*0.389}" upper="${pi*0.389}" />
+      <limit velocity="4.8" effort="30" lower="${-pi*0.5}" upper="${pi*0.5}" />
       <dynamics damping="0.1" />
     </joint>

Commit message: 각도 업데이트

File: avatar_description/ros2_control/follower.ros2_control.xacro (robot description, xacro)
@@ -299,21 +299,4 @@
           <param name="Operating Mode">3</param>
           <param name="Return Delay Time">0</param>
-          <param name="Min Position Limit">1024</param>
-          <param name="Max Position Limit">3140</param>
-          <param name="Position P Gain">1000</param>
-          <param name="Position I Gain">0</param>
-          <param name="Position D Gain">1000</param>
-          <param name="Profile Velocity">50</param>
-          <param name="Profile Acceleration">25</param>
-        </gpio>
-        <gpio name="dxl22">
-          <param name="type">dxl</param>
-          <param name="ID">22</param>
-          <command_interface name="Goal Position"/>
-          <state_interface name="Present Position"/>
-          <state_interface name="Present Velocity"/>
-          <param name="Drive Mode">4</param>
-          <param name="Operating Mode">3</param>
-          <param name="Return Delay Time">0</param>
           <param name="Min Position Limit">548</param>
           <param name="Max Position Limit">3548</param>
@@ -324,7 +307,7 @@
           <param name="Profile Acceleration">25</param>
         </gpio>
-        <gpio name="dxl23">
-          <param name="type">dxl</param>
-          <param name="ID">23</param>
+        <gpio name="dxl22">
+          <param name="type">dxl</param>
+          <param name="ID">22</param>
           <command_interface name="Goal Position"/>
           <state_interface name="Present Position"/>
@@ -341,4 +324,21 @@
           <param name="Profile Acceleration">25</param>
         </gpio>
+        <gpio name="dxl23">
+          <param name="type">dxl</param>
+          <param name="ID">23</param>
+          <command_interface name="Goal Position"/>
+          <state_interface name="Present Position"/>
+          <state_interface name="Present Velocity"/>
+          <param name="Drive Mode">4</param>
+          <param name="Operating Mode">3</param>
+          <param name="Return Delay Time">0</param>
+          <param name="Min Position Limit">1024</param>
+          <param name="Max Position Limit">3072</param>
+          <param name="Position P Gain">1000</param>
+          <param name="Position I Gain">0</param>
+          <param name="Position D Gain">1000</param>
+          <param name="Profile Velocity">50</param>
+          <param name="Profile Acceleration">25</param>
+        </gpio>
         <gpio name="dxl24">
           <param name="type">dxl</param>
@@ -350,5 +350,5 @@
           <param name="Operating Mode">3</param>
           <param name="Return Delay Time">0</param>
-          <param name="Min Position Limit">1024</param>
+          <param name="Min Position Limit">2048</param>
           <param name="Max Position Limit">3072</param>
           <param name="Position P Gain">1000</param>

File: avatar_description/urdf/follower/follower_arm.urdf.xacro (robot description, xacro)
@@ -356,5 +356,5 @@
       <child link="${prefix}right_link1_1"/>
       <axis xyz="-0.0 -1.0 0.0"/>
-      <limit velocity="4.8" effort="30" lower="${-pi*2.0}" upper="${pi*2.0}" />
+      <limit velocity="4.8" effort="30" lower="${-pi*0.7323888889}" upper="${pi*0.7323888889}" />
       <dynamics damping="0.1" />
     </joint>
@@ -364,5 +364,5 @@
       <child link="${prefix}right_link2_1"/>
       <axis xyz="1.0 -0.0 0.0"/>
-      <limit velocity="4.8" effort="30" lower="${-pi*2.0}" upper="${pi*2.0}" />
+      <limit velocity="4.8" effort="30" lower="${-pi*0.4550555556}" upper="${pi*0.0253888889}" />
       <dynamics damping="0.1" />
     </joint>
@@ -372,5 +372,5 @@
       <child link="${prefix}right_link3_1"/>
       <axis xyz="0.0 -0.0 -1.0"/>
-      <limit velocity="4.8" effort="30" lower="${-pi*2.0}" upper="${pi*2.0}" />
+      <limit velocity="4.8" effort="30" lower="${-pi*0.5}" upper="${pi*0.5}" />
       <dynamics damping="0.1" />
     </joint>
@@ -380,5 +380,5 @@
       <child link="${prefix}right_link4_1"/>
       <axis xyz="0.0 -1.0 -0.0"/>
-      <limit velocity="4.8" effort="30" lower="${-pi*0.5}" upper="${pi*0.5}" />
+      <limit velocity="4.8" effort="30" lower="${-pi*0.0}" upper="${pi*0.5}" />
       <dynamics damping="0.1" />
     </joint>
@@ -396,5 +396,5 @@
       <child link="${prefix}right_link6_1"/>
       <axis xyz="0.0 -1.0 0.0"/>
-      <limit velocity="4.8" effort="30" lower="${-pi*0.389}" upper="${pi*0.389}" />
+      <limit velocity="4.8" effort="30" lower="${-pi*0.3866666667}" upper="${pi*0.3866666667}" />
       <dynamics damping="0.1" />
     </joint>
@@ -404,5 +404,5 @@
       <child link="${prefix}right_link_gripper_1"/>
       <axis xyz="1.0 -0.0 -0.0"/>
-      <limit velocity="4.8" effort="30" lower="${-pi*2.0}" upper="${pi*2.0}" />
+      <limit velocity="4.8" effort="30" lower="${-pi*0.0}" upper="${pi*0.6210555556}" />
       <dynamics damping="0.1" />
     </joint>
@@ -412,5 +412,5 @@
       <child link="${prefix}left_link1_1"/>
       <axis xyz="0.0 1.0 0.0"/>
-      <limit velocity="4.8" effort="30" lower="${-pi*0.5}" upper="${pi*0.5}" />
+      <limit velocity="4.8" effort="30" lower="${-pi*0.7323888889}" upper="${pi*0.7323888889}" />
       <dynamics damping="0.1" />
     </joint>
@@ -420,5 +420,5 @@
       <child link="${prefix}left_link2_1"/>
       <axis xyz="1.0 -0.0 -0.0"/>
-      <limit velocity="4.8" effort="30" lower="${-pi*2.0}" upper="${pi*2.0}" />
+      <limit velocity="4.8" effort="30" lower="${-pi*0.0253888889}" upper="${pi*0.4550555556}" />
       <dynamics damping="0.1" />
     </joint>
@@ -428,5 +428,5 @@
       <child link="${prefix}left_link3_1"/>
       <axis xyz="0.0 -0.0 -1.0"/>
-      <limit velocity="4.8" effort="30" lower="${-pi*2.0}" upper="${pi*2.0}" />
+      <limit velocity="4.8" effort="30" lower="${-pi*0.5}" upper="${pi*0.5}" />
       <dynamics damping="0.1" />
     </joint>
@@ -436,5 +436,5 @@
       <child link="${prefix}left_link4_1"/>
       <axis xyz="-0.0 1.0 0.0"/>
-      <limit velocity="4.8" effort="30" lower="${-pi*0.5}" upper="${pi*0.5}" />
+      <limit velocity="4.8" effort="30" lower="${-pi*0.5}" upper="${pi*0.0}" />
       <dynamics damping="0.1" />
     </joint>
@@ -452,5 +452,5 @@
       <child link="${prefix}left_link6_1"/>
       <axis xyz="-0.0 1.0 -0.0"/>
-      <limit velocity="4.8" effort="30" lower="${-pi*0.389}" upper="${pi*0.389}" />
+      <limit velocity="4.8" effort="30" lower="${-pi*0.3866666667}" upper="${pi*0.3866666667}" />
       <dynamics damping="0.1" />
     </joint>
@@ -460,5 +460,5 @@
       <child link="${prefix}left_link_gripper_1"/>
       <axis xyz="1.0 -0.0 -0.0"/>
-      <limit velocity="4.8" effort="30" lower="${-pi*2.0}" upper="${pi*2.0}" />
+      <limit velocity="4.8" effort="30" lower="${-pi*0.6210555556}" upper="${pi*0.0}" />
       <dynamics damping="0.1" />
     </joint>
@@ -468,5 +468,5 @@
       <child link="${prefix}neck_link1_1"/>
       <axis xyz="0.0 1.0 -0.0"/>
-      <limit velocity="4.8" effort="30" lower="${-pi*2.0}" upper="${pi*2.0}" />
+      <limit velocity="4.8" effort="30" lower="${-pi*0.1620555556}" upper="${pi*0.1620555556}" />
       <dynamics damping="0.1" />
     </joint>
@@ -476,5 +476,5 @@
       <child link="${prefix}neck_link2_1"/>
       <axis xyz="0.0 0.0 1.0"/>
-      <limit velocity="4.8" effort="30" lower="${-pi*0.5}" upper="${pi*0.5}" />
+      <limit velocity="4.8" effort="30" lower="${-pi*0.2441111111}" upper="${pi*0.2441111111}" />
       <dynamics damping="0.1" />
     </joint>
